File: pocket-reform-motherboard/pocket-reform-motherboard.sch (KiCad schematic (older format))
At the start: 20 parts, among them J1 PWR, J2 Micro_SD_Card_Det, J3 USB_C_Receptacle, J4 AudioJack4, J5 USB_C_Receptacle, J6 USBINT, J7 HDMI_D_1.4, J8 SIM_Card, U1 reform2-som-connector, U2 MPCIE-Socket-reform-motherboa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, U3 TUSB4041I, U4 WM8960, U6 MPCIE-Socket-reform-motherboa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

Commit message: motherboard: first routing
Parts:
- removed J5: USB_C_Receptacle, Connector_USB:USB_C_Receptacle_Amphenol_12401548E4-2A_CircularHoles, symbol Connector:USB_C_Receptacle
- removed TP1, TP2: TestPoint_2Pole, footprints:MOLEX_48099-5701, symbol Connector:TestPoint_2Pole
- removed U2, U6: MPCIE-Socket-reform-motherboard-rescue, footprints:MOLEX_67910-5700, symbol reform2-motherboard-rescue:MPCIE-Socket-reform-motherboard-rescue
- added C1, C2: 18pF, Capacitor_SMD:C_0603_1608Metric, symbol reform2-motherboard-rescue:C_Small-reform-motherboard-rescue
- added C123, C124, C126, C83: 47uF, Capacitor_SMD:C_0603_1608Metric, symbol Device:C_Small
- added C152, C153, C52, C58: 10nF, Capacitor_SMD:C_0603_1608Metric, symbol Device:C_Small
- added C53, C54, C55, C59, C60, C61: 0.1uF, Capacitor_SMD:C_0603_1608Metric, symbol Device:C_Small
- added D1, D23: LED_NVME, LED_SMD:LED_0603_1608Metric, symbol Device:LED_Small
- added FB3, FB4: 100@100MHz 3A, Inductor_SMD:L_0603_1608Metric, symbol Device:Ferrite_Bead_Small
- added J10, J9: 1-2199230-6, footprints:TE_1-2199230-6, symbol reform2:1-2199230-6
- added J5: USB_C_Receptacle_USB2.0, Type-C:HRO-TYPE-C-31-M-12, symbol Connector:USB_C_Receptacle_USB2.0
- added R1, R110: 1k, Resistor_SMD:R_0603_1608Metric, symbol Device:R_Small
- added R104, R105, R106, R107, R108, R109, R2, R3, R39, R4, R5, R6, R7: 0, Resistor_SMD:R_0603_1608Metric, symbol Device:R_Small
- added R122, R37, R38, R40: 1.5k, Resistor_SMD:R_0603_1608Metric, symbol Device:R_Small
- added R123, R148, R198, R199: 49.9, Resistor_SMD:R_0603_1608Metric, symbol Device:R_Small
- added R160: 100k, Resistor_SMD:R_0603_1608Metric, symbol Device:R_Small
- added R36: 475, Resistor_SMD:R_0603_1608Metric, symbol Device:R_Small
- added R8: 1M, Resistor_SMD:R_0603_1608Metric, symbol reform2-motherboard-rescue:R_Small-reform-motherboard-rescue
- added U23: IDT5V41066, Package_SO:TSSOP-20_4.4x6.5mm_P0.65mm, symbol reform2:IDT5V41066
- added Y1: 25MHz, Crystal:Crystal_SMD_Abracon_ABM8G-4Pin_3.2x2.5mm, symbol Device:Crystal_GND24_Small
Connections:
- net +3V3: now also FB3.1, FB4.1
- net GND: now also C1.2, C123.2, C124.2, C126.2, C152.2, C153.2, C2.2, C52.2, C53.2, C54.2, C55.2, C58.2, C59.2, C60.2, C61.2, C83.2, J10.1, J10.15, J10.21, J10.27, J10.3, J10.33, J10.39, J10.45, J10.51, J10.57, J10.71, J10.73, J10.75, J10.9, J10.S1 (SHIELD), J10.S2 (SHIELD), J9.1, J9.15, J9.21, J9.27, J9.3, J9.33, J9.39, J9.45, J9.51, J9.57, J9.71, J9.73, J9.75, J9.9, J9.S1 (SHIELD), J9.S2 (SHIELD), R104.2, R105.2, R106.2, R107.2, R108.2, R109.2, R123.1, R148.1, R198.1, R199.1, R2.2, R3.2, R36.1, R39.1, R4.2, R5.2, R6.2, R7.2, U23.16 (GNDODA), U23.9 (GNDXD), Y1.2, Y1.4
- net USB12_DN: no longer J3.A7 (D-), J3.B7 (D-)
- net USB12_DP: no longer J3.A6 (D+), J3.B6 (D+)
- net USB2_DN: now also J3.A7 (D-), J3.B7 (D-)
- net USB2_DP: now also J3.A6 (D+), J3.B6 (D+)
- new net: D23.1 (K), J10.10
- new net: D23.2 (A), R110.2
- new net: C124.1, C126.1, C58.1, C59.1, C60.1, C61.1, FB4.2, J10.12, J10.14, J10.16, J10.18, J10.2, J10.4, J10.70, J10.72, J10.74, R110.1
- new net: J10.11, R107.1
- new net: J10.13, R104.1
- new net: J10.23, R108.1
- new net: J10.25, R105.1
- new net: J10.35, R109.1
- new net: J10.37, R106.1
- new net: C123.1, C52.1, C53.1, C54.1, C55.1, C83.1, FB3.2, J9.12, J9.14, J9.16, J9.18, J9.2, J9.4, J9.70, J9.72, J9.74, R1.1
- new net: R36.2, U23.10 (IREF)
- new net: C152.1, C153.1, R122.1, R37.1, R38.1, R40.1, U23.1 (VDDXD), U23.15 (VDDODA)
- new net: R37.2, U23.2 (S0)
- new net: R38.2, U23.3 (S1)
- new net: R40.2, U23.7 (~PD)
- new net: R39.2, U23.4 (S2)
- new net: J10.55, R198.2, U23.14 (CLKC_P)
- new net: R122.2, U23.8 (OE)
- new net: J5.A1 (GND), J5.A12 (GND), J5.B1 (GND), J5.B12 (GND)
- new net: J5.A4 (VBUS), J5.A9 (VBUS), J5.B4 (VBUS), J5.B9 (VBUS)
- new net: D1.1 (K), J9.10
- new net: J9.11, R2.1
- new net: J9.13, R3.1
- new net: J9.23, R4.1
- new net: J9.25, R5.1
- new net: J9.35, R6.1
- new net: J9.37, R7.1
- new net: D1.2 (A), R1.2
- new net M2_CLKREQn: J10.52, J9.52
- new net M2_SMB_ALERTn: J10.44
- new net M2_SMB_CLK: J10.40
- new net M2_SMB_DATA: J10.42
- new net PCICLKGEN_XI: C2.1, R8.2, U23.5 (X1), Y1.3
- new net PCICLKGEN_XO: C1.1, R8.1, U23.6 (X2), Y1.1
- new net PCIE2_CLK_N: J9.55, R148.2, U23.11 (CLKD_N)
- new net PCIE2_CLK_P: J9.53, R123.2, U23.12 (CLKD_P)
- new net PCIE2_RESETn: J10.50, J9.50
- new net PCIE2_RX_N: J10.41, J9.41
- new net PCIE2_RX_P: J10.43, J9.43
- new net PCIE2_TX_N: J10.47, J9.49
- new net PCIE2_TX_P: J10.49, J9.47
- new net RCLKC_N: J10.53, R199.2, U23.13 (CLKC_N)
- no-connect marks 48 -> 112
Other:
- note added: "1-2199230-5"
- note added: "2280 formfactor"
- note added: "M Key 42H M.2"
- note added: "M.2 footprint by takigama https://github.com/takigama/KiCADComponents"
- note added: "PERn1"
- note added: "PERn2"
- note added: "PERn3"
- note added: "PERp1"
- note added: "PERp2"
- note added: "PERp3"
- note added: "PETn1"
- note added: "PETn2"
- note added: "PETn3"
- note added: "PETp1"
- note added: "PETp2"
- note added: "PETp3"
- note added: "Refclk Generator"
- note added: "TODO: B KEY"
- note added: "TODO: mux!"
- note added: "TODO: obsolete chip?"
- note added: "TX caps are on the SoM"
- note added: "Thanks to Austin @ ZII for\nlane wrangling info!"
- note added: "https://cdn.techship.com//uploads/images/3421/11312_210415.png"
- note added: "https://github.com/ai03-2725/Type-C.pretty"
- note removed: "TODO: UIM"
- note removed: "TODO: import the audio filters etc"
- moved on the sheet: GFX1, H1, H2, H3, H4, J1, J2, J3, J4, J6, J7, J8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
