File: pocket-reform-motherboard/pocket-reform-motherboard.kicad_sch (KiCad schematic)
At the start: 278 parts

Commit message: motherboard: first routing
Parts:
- removed C1, C3: (no value), symbol Device:C_Small
- removed D2: (no value), symbol Device:D_Schottky
- removed D3: (no value), symbol Device:D_Zener_Small_Filled
- removed Q1: (no value), symbol reform2:Si7465DP
- removed R2, R3: (no value), symbol Device:R_Small
- added D2: PMEG3050EP,115, Diode_SMD:D_SOD-128, symbol Device:D_Schottky_Small_Filled
- added J16, J17: Conn_01x03, Connector_PinHeader_2.54mm:PinHeader_1x03_P2.54mm_Vertical, symbol Connector_Generic:Conn_01x03
- BT1: value (none) -> V364; footprint (none) -> Battery:BatteryHolder_Keystone_2998_1x6.8mm
- C10, C20, C26, C34, C36, C9: value (none) -> 1uF; footprint (none) -> Capacitor_SMD:C_0603_1608Metric
- C11, C12, C18, C19, C52, C58, C7, C8: value (none) -> 10nF; footprint (none) -> Capacitor_SMD:C_0603_1608Metric
- C123, C124, C126, C14, C83: value (none) -> 47uF; footprint (none) -> Capacitor_SMD:C_0603_1608Metric
- C13: value (none) -> 12pF; footprint (none) -> Capacitor_SMD:C_0603_1608Metric
- C15, C16: value (none) -> 330uF; footprint (none) -> Capacitor_SMD:CP_Elec_6.3x5.4
- C17, C2, C39, C4, C5, C6, C65: value (none) -> 10uF; footprint (none) -> Capacitor_SMD:C_0603_1608Metric
- C21, C23: value (none) -> 18pF; footprint (none) -> Capacitor_SMD:C_0603_1608Metric
- C22, C24: value (none) -> 27pF; footprint (none) -> Capacitor_SMD:C_0603_1608Metric
- C25, C27, C28, C29, C30, C31, C32, C33, C35, C38, C40, C41, C42, C43, C44, C45, C46, C47, C48, C49, C53, C54, C55, C59, C60, C61, C63, C64, C66, C72, C73, C77, C85, C86, C87, C88, C89, C90, C91, C92, C93: value (none) -> 0.1uF; footprint (none) -> Capacitor_SMD:C_0603_1608Metric
- C37: value (none) -> 1nF; footprint (none) -> Capacitor_SMD:C_0603_1608Metric
- C51, C67: value (none) -> 10uF
- C68: value (none) -> 0.1uF
- D1: value (none) -> LED_MODEM; footprint (none) -> LED_SMD:LED_0603_1608Metric
- D10: value (none) -> 19-337/R6GHBHC-A01/2T; footprint (none) -> footprints:LED_19-337_R6GHBHC-A01_2T
- D11: value (none) -> SS54?; footprint (none) -> Diode_SMD:D_SMA
- D12: value (none) -> SD0603S040S0R2; footprint (none) -> Diode_SMD:D_0603_1608Metric
- D23: value (none) -> LED_NVME; footprint (none) -> LED_SMD:LED_0603_1608Metric
- D4, D5, D6: value (none) -> PMEG3050EP,115; footprint (none) -> Diode_SMD:D_SOD-128
- D7: value (none) -> BZX84-C5V6,215; footprint (none) -> Diode_SMD:D_SOD-323
- D8, D9: value (none) -> LED_Small; footprint (none) -> LED_SMD:LED_0603_1608Metric
- FB1: value (none) -> 220@100MHz 1.4A; footprint (none) -> Inductor_SMD:L_0603_1608Metric
- FB3, FB4, FB8: value (none) -> 100@100MHz 3A; footprint (none) -> Inductor_SMD:L_0603_1608Metric
- GFX1: value (none) -> MountingHole; footprint (none) -> footprints:pocket-reform
- H1, H2, H3, H4: value (none) -> MountingHole_Pad; footprint (none) -> MountingHole:MountingHole_2.2mm_M2_DIN965_Pad
- J1: value (none) -> CHARGER; footprint (none) -> Connector_JST:JST_PH_S9B-PH-SM4-TB_1x09-1MP_P2.00mm_Horizontal
- J10: value (none) -> 1-2199230-6; footprint (none) -> footprints:TE_1-2199230-6
- J11: value (none) -> Conn_01x33; footprint (none) -> Connector_FFC-FPC:Hirose_FH12-33S-0.5SH_1x33-1MP_P0.50mm_Horizontal
- J12: value (none) -> 2199230-5; footprint (none) -> footprints:TE_2199230-5
- J13: value (none) -> FH35C-31S-0.3HW(50); footprint (none) -> footprints:TE_3-2328724-1
- J14, J3: value (none) -> USB_C_Receptacle; footprint (none) -> Connector_USB:USB_C_Receptacle_Amphenol_12401548E4-2A_CircularHoles
- J15: value (none) -> Conn_01x02; footprint (none) -> Connector_JST:JST_GH_SM02B-GHS-TB_1x02-1MP_P1.25mm_Horizontal
- J2: value (none) -> DM3AT-SF-PEJM5; footprint (none) -> footprints:DM3AT-SF-PEJM5; LCSC (none) -> C114218
- J4: value (none) -> 09452812561; footprint (none) -> footprints:09452812561; Manufacturer (none) -> HARTING; Manufacturer_Name HARTING -> (none)
- J5: value (none) -> SYSCTL; footprint (none) -> Connector_JST:JST_PH_S4B-PH-SM4-TB_1x04-1MP_P2.00mm_Horizontal
- J6: value (none) -> USB_INT1; footprint (none) -> Connector_JST:JST_PH_S4B-PH-SM4-TB_1x04-1MP_P2.00mm_Horizontal
- J7: value (none) -> HDMI_D_1.4; footprint (none) -> Connector_HDMI:HDMI_Micro-D_Molex_46765-0x01
- J8: value (none) -> SIM_Card; footprint (none) -> footprints:MOLEX_78800-0001
- J9: value (none) -> USB_C_Receptacle_USB2.0; footprint (none) -> Connector_USB:USB_C_Receptacle_HRO_TYPE-C-31-M-12
- L1: value (none) -> 22uH; footprint (none) -> Inductor_SMD:L_Taiyo-Yuden_NR-30xx
- L2: value (none) -> 2.2uH; footprint (none) -> Inductor_SMD:L_1210_3225Metric
- L3, L4: value (none) -> 15uH; footprint (none) -> Inductor_SMD:L_Vishay_IHLP-4040; Manufacturer (none) -> Vishay
- L5, L6: footprint Inductor_SMD:L_1210_3225Metric -> Inductor_SMD:L_Taiyo-Yuden_NR-30xx; LCSC (none) -> C223122; Manufacturer Murata -> Taiyo Yuden; Manufacturer_No LQH32PB150MN0L -> NRH3012T150MN
- MK1: value (none) -> MP23ABS1TR; footprint (none) -> footprints:MIC_MP23ABS1TR
- R1, R110, R29, R34, R35, R36, R58, R60, R61: value (none) -> 1k; footprint (none) -> Resistor_SMD:R_0603_1608Metric
- R10, R27, R55: value (none) -> 200k; footprint (none) -> Resistor_SMD:R_0603_1608Metric
- R100, R97, R98, R99: value (none) -> 47k; footprint (none) -> Resistor_SMD:R_0603_1608Metric
- R101, R102, R103, R104, R105, R106, R107, R108, R109, R11, R111, R12, R13, R4, R44, R45, R46, R49, R5, R50, R51, R67, R71, R81, R83, R84, R9: value (none) -> 0; footprint (none) -> Resistor_SMD:R_0603_1608Metric
- R14: value (none) -> 280k; footprint (none) -> Resistor_SMD:R_0603_1608Metric
- R15, R17, R22, R30, R32, R38, R52, R54, R56, R68, R75, R85, R96: value (none) -> 10k; footprint (none) -> Resistor_SMD:R_0603_1608Metric
- R16: value (none) -> 3.16k; footprint (none) -> Resistor_SMD:R_0603_1608Metric
- R18: value (none) -> 5.83k; footprint (none) -> Resistor_SMD:R_0603_1608Metric
- R19: value (none) -> 1.3M; footprint (none) -> Resistor_SMD:R_0603_1608Metric
- R198, R199, R65, R66: value (none) -> 49.9; footprint (none) -> Resistor_SMD:R_0603_1608Metric
- R20: value (none) -> 300k; footprint (none) -> Resistor_SMD:R_0603_1608Metric
- R21: value (none) -> 1M; footprint (none) -> Resistor_SMD:R_0603_1608Metric
- R23, R62, R63, R64: value (none) -> DNP; footprint (none) -> Resistor_SMD:R_0603_1608Metric
- R24, R25, R26, R57, R59, R89, R93: value (none) -> 4.7k; footprint (none) -> Resistor_SMD:R_0603_1608Metric
- R28: value (none) -> 120k; footprint (none) -> Resistor_SMD:R_0603_1608Metric
- R31, R33: value (none) -> 36k; footprint (none) -> Resistor_SMD:R_0603_1608Metric
- R37, R39, R40, R41: value (none) -> 75 1%; footprint (none) -> Resistor_SMD:R_0603_1608Metric
- R47, R48: value (none) -> 27.4; footprint (none) -> Resistor_SMD:R_0603_1608Metric
- R53: value (none) -> 12k 1%; footprint (none) -> Resistor_SMD:R_0603_1608Metric
- R6, R69, R7, R8, R87: value (none) -> 100k; footprint (none) -> Resistor_SMD:R_0603_1608Metric
- R70: footprint (none) -> Resistor_SMD:R_0603_1608Metric
- R72: value (none) -> 2k2; footprint (none) -> Resistor_SMD:R_0603_1608Metric
- R90: value (none) -> 27k; footprint (none) -> Resistor_SMD:R_0603_1608Metric
- SW1: value (none) -> SW_DIP_x01; footprint (none) -> Button_Switch_SMD:SW_DIP_SPSTx01_Slide_Omron_A6S-110x_W8.9mm_P2.54mm
- SW2: value (none) -> RESET; footprint (none) -> Button_Switch_SMD:SW_Push_1P1T_NO_CK_KMR2
- TP1: value (none) -> PRTCTL1; footprint (none) -> TestPoint:TestPoint_Pad_D1.0mm
- TP2: value (none) -> PRTCTL3; footprint (none) -> TestPoint:TestPoint_Pad_D1.0mm
- TP3: value (none) -> PRTCTL2; footprint (none) -> TestPoint:TestPoint_Pad_D1.0mm
- TP4: value (none) -> PRTCTL4; footprint (none) -> TestPoint:TestPoint_Pad_D1.0mm
- TP5, TP6: value (none) -> TestPoint; footprint (none) -> TestPoint:TestPoint_Pad_D1.0mm
- TR1: value (none) -> TG111-MSC13LF; footprint (none) -> Transformer_SMD:Transformer_Ethernet_HALO_TG111-MSC13
- U1: value (none) -> reform2-som-connector; footprint (none) -> footprints:TE_1473149-4
- U10: value (none) -> W25Q32JVSS; footprint (none) -> Package_SO:SOIC-8_5.23x5.23mm_P1.27mm
- U11: value (none) -> PCF8523T; footprint (none) -> Package_SO:SOIC-8_3.9x4.9mm_P1.27mm
- U12: value (none) -> AP22815; footprint (none) -> Package_TO_SOT_SMD:SOT-23-5
- U13: value (none) -> TXS0108EPW; footprint (none) -> Package_SO:TSSOP-20_4.4x6.5mm_P0.65mm
- U14: value (none) -> SN74AVC1T45; footprint (none) -> Package_TO_SOT_SMD:SOT-23-6
- U15, U16, U19, U20, U21, U22: value (none) -> TPD4E02B04DQA; footprint (none) -> Package_SON:USON-10_2.5x1.0mm_P0.5mm
- U17: value (none) -> TPD12S521; footprint (none) -> footprints:TSSOP50P640X120-38N
- U18: value (none) -> TLV320AIC3100; footprint (none) -> Package_DFN_QFN:VQFN-32-1EP_5x5mm_P0.5mm_EP3.5x3.5mm
- U2: value (none) -> MAX1837EUT33+T; footprint (none) -> Package_TO_SOT_SMD:SOT-23-6
- U23: value (none) -> FUSB302BMPX; footprint (none) -> Package_DFN_QFN:WQFN-14-1EP_2.5x2.5mm_P0.5mm_EP1.45x1.45mm
- U3: value (none) -> LM3674MFX-ADJ/NOPB; footprint (none) -> Package_TO_SOT_SMD:SOT-23-5
- U4: value (none) -> TLV1117-18; footprint (none) -> Package_TO_SOT_SMD:SOT-223
- U5, U6: value (none) -> TPS5450DDAR; footprint (none) -> Package_SO:TI_SO-PowerPAD-8_ThermalVias
- U7: value (none) -> CN301; footprint (none) -> Package_TO_SOT_SMD:SOT-23-5
- U8: value (none) -> RP2040; footprint (none) -> footprints:RP2040-QFN-56
- U9: value (none) -> USB7002/KDX; footprint (none) -> footprints:QFN40P1200X1200X90-101N
- Y1: value (none) -> 25MHz; footprint (none) -> Crystal:Crystal_SMD_Abracon_ABM8G-4Pin_3.2x2.5mm
- Y2: value (none) -> 12MHz 18pF; footprint (none) -> Crystal:Crystal_SMD_3225-4Pin_3.2x2.5mm
- Y3: value (none) -> 32.768 kHz; footprint (none) -> Crystal:Crystal_SMD_3215-2Pin_3.2x1.5mm
Connections:
- net GND: now also J2.10 (DET_A), D2.2 (A), J16.3 (Pin_3), J17.3 (Pin_3)
- net IMX_UART1_RX: now also J16.2 (Pin_2)
- net IMX_UART1_TX: now also J16.1 (Pin_1)
- net IMX_UART2_RX: now also J17.2 (Pin_2)
- net IMX_UART2_TX: now also J17.1 (Pin_1)
- net VCC: now also J1.1 (Pin_1), J1.2 (Pin_2), D2.1 (K)
- no-connect marks 194 -> 193
Other:
- note added: "Keystone 2998 C238096"
- note added: "NRH3012T220MN"
- note added: "Needs inrush limiter on charger board!"
- note added: "ROQANG RVT0J331M0605"
- note added: "SFV33R-1STBE1HLF"
- note added: "Serial Ports"
- note removed: "DM3CS-SF"
- note removed: "Inrush Current Limiter by Zoé"
- moved on the sheet: C14, C6, J11, J13

Commit message: motherboard: routing snapshot
Parts:
- added C1, C100, C3, C70, C71, C74, C75, C79, C80, C81, C84, C94, C95, C96, C97, C98, C99: 0.1uF, Capacitor_SMD:C_0402_1005Metric, symbol Device:C_Small
- C25, C27, C28, C29, C30, C31, C32, C33, C35, C38, C40, C41, C42, C43, C44, C45, C46, C47, C48, C49, C50, C53, C54, C55, C57, C59, C60, C61, C62, C63, C64, C66, C68, C69, C72, C73, C76, C77, C78, C85, C86, C87, C88, C89, C90, C91, C92, C93: footprint Capacitor_SMD:C_0603_1608Metric -> Capacitor_SMD:C_0402_1005Metric
- R10, R15, R17, R22, R24, R25, R26, R27, R30, R32, R38, R52, R54, R55, R56, R57, R59, R68, R75, R85, R89, R93, R96: footprint Resistor_SMD:R_0603_1608Metric -> Resistor_SMD:R_0402_1005Metric
- U15, U16, U19, U20, U21, U22: symbol Power_Protection:TPD4E02B04DQA -> pocket-reform:TPD4E02B04DQA_RT
Connections:
- net +1V2: now also C1.1, C100.1, C70.1, C74.1, C79.1, C81.1, C94.1, C96.1, C98.1
- net +3V3: now also C3.1, C71.1, C75.1, C80.1, C84.1, C95.1, C97.1, C99.1
- net GND: now also C1.2, C100.2, C3.2, C70.2, C71.2, C74.2, C75.2, C79.2, C80.2, C81.2, C84.2, C94.2, C95.2, C96.2, C97.2, C98.2, C99.2
- net USBH_1A_RXN: now also U20.10 (IO1)
- net USBH_1A_RXP: now also U20.9 (IO2)
- net USBH_1B_RXN: now also U22.10 (IO1)
- net USBH_1B_RXP: now also U22.9 (IO2)
- net USBH_1_DN: now also U16.7 (IO3)
- net USBH_1_DP: now also U16.6 (IO4)
- net USBH_2A_RXN: now also U19.10 (IO1)
- net USBH_2A_RXP: now also U19.9 (IO2)
- net USBH_2B_RXN: now also U21.10 (IO1)
- net USBH_2B_RXP: now also U21.9 (IO2)
- net USBH_2_DN: now also U15.7 (IO3)
- net USBH_2_DP: now also U15.6 (IO4)
- net USBH_1A_AC_TXP: now reaches C88.1, J3.A2 (TX1+), U20.5 (IO4)
- net USBH_1A_AC_TXP: now also U20.6 (IO4)
- net USBH_1A_AC_TXN: now reaches C85.1, J3.A3 (TX1-), U20.4 (IO3)
- net USBH_1A_AC_TXN: now also U20.7 (IO3)
- net at J3.A5 (CC1), R83.1, U16.1 (IO1): now also U16.10 (IO1)
- net USBH_1B_AC_TXP: now reaches C89.1, J3.B2 (TX2+), U22.5 (IO4)
- net USBH_1B_AC_TXP: now also U22.6 (IO4)
- net USBH_1B_AC_TXN: now reaches C86.1, J3.B3 (TX2-), U22.4 (IO3)
- net USBH_1B_AC_TXN: now also U22.7 (IO3)
- net at J3.B5 (CC2), R84.1, U16.2 (IO2): now also U16.9 (IO2)
- net USBH_2B_AC_TXN: now reaches C91.1, J14.B3 (TX2-), U21.4 (IO3)
- net USBH_2B_AC_TXN: now also U21.7 (IO3)
- net USBH_2A_AC_TXN: now reaches C90.1, J14.A3 (TX1-), U19.4 (IO3)
- net USBH_2A_AC_TXN: now also U19.7 (IO3)
- net at J14.A5 (CC1), R101.2, R111.1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: now also U15.10 (IO1)
- net at J14.B5 (CC2), R102.2, R103.1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: now also U15.9 (IO2)
- net USBH_2B_AC_TXP: now reaches C93.1, J14.B2 (TX2+), U21.5 (IO4)
- net USBH_2B_AC_TXP: now also U21.6 (IO4)
- net USBH_2A_AC_TXP: now reaches C92.1, J14.A2 (TX1+), U19.5 (IO4)
- net USBH_2A_AC_TXP: now also U19.6 (IO4)
Other:
- note added: "alt: USB5534B-5000JZX"
- note added: "https://www.microchipdirect.com/product/USB7002T-I/KDXVAO?productLoaded=true"

Commit message: snapshot before replacing usb7002
Other:
- note added: "TODO: TUSB8040 needs up to 1A, USB7002 up to 500mA"
Changed lines of the file:
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@@
+    (effects (font (size 1.27 1.27)) (justify left bottom))
+  )
+  (text "TODO: TUSB8040 needs up to 1A,\nUSB7002 up to 500mA"
+    (at 200.66 254 0)
     (effects (font (size 1.27 1.27)) (justify left bottom))
   )

Commit message: routing snapshot with TUSB8040
Parts:
- removed R101, R102: 0, Resistor_SMD:R_0603_1608Metric, symbol Device:R_Small
- removed R27, R55: 200k, Resistor_SMD:R_0402_1005Metric, symbol Device:R_Small
- removed R30, R32, R52, R54: 10k, Resistor_SMD:R_0402_1005Metric, symbol Device:R_Small
- removed R31, R33: 36k, Resistor_SMD:R_0603_1608Metric, symbol Device:R_Small
- removed R53: 12k 1%, Resistor_SMD:R_0603_1608Metric, symbol Device:R_Small
- removed TP1: PRTCTL1, TestPoint:TestPoint_Pad_D1.0mm, symbol Connector:TestPoint
- removed TP2: PRTCTL3, TestPoint:TestPoint_Pad_D1.0mm, symbol Connector:TestPoint
- removed TP3: PRTCTL2, TestPoint:TestPoint_Pad_D1.0mm, symbol Connector:TestPoint
- removed TP4: PRTCTL4, TestPoint:TestPoint_Pad_D1.0mm, symbol Connector:TestPoint
- removed U9: USB7002/KDX, footprints:QFN40P1200X1200X90-101N, symbol USB7002_KDX:USB7002/KDX
- added C101: 0.1uF, Capacitor_SMD:C_0402_1005Metric, symbol Device:C_Small
- added FB7: 220@100MHz 1.4A, Inductor_SMD:L_0603_1608Metric, symbol Device:FerriteBead_Small
- added R2: 1M, Resistor_SMD:R_0603_1608Metric, symbol Device:R_Small
- added R3: 90.9K 1%, Resistor_SMD:R_0603_1608Metric, symbol Device:R_Small
- added U9: TUSB8040PFP, footprints:QFP50P1400X1400X120-81N, symbol pocket-reform:TUSB8040PFP
- C100, C98: value 0.1uF -> 10uF
- C95, C97, C99: value 0.1uF -> 1uF
- R22: value 10k -> R_Small
- R23: value DNP -> 9.09K 1%
- R24, R25, R26: value 4.7k -> 10k; footprint Resistor_SMD:R_0402_1005Metric -> Resistor_SMD:R_0603_1608Metric
- Y1: value 25MHz -> 24MHz
Connections:
- net +1V2: now also C3.1, C71.1, C101.1, U9.1 (VDD11), U9.10 (VDD11), U9.11 (VDD11), U9.16 (VDD11), U9.20 (VDD11), U9.26 (VDD11), U9.32 (VDD11), U9.37 (VDD11), U9.42 (VDD11), U9.46 (VDD11), U9.5 (VDD11), U9.51 (VDD11), U9.52 (VDD11), U9.57 (VDD11), U9.61 (VDD11), U9.67 (VDD11), U9.71 (VDD11)
- net +3V3: now also FB7.2; no longer C3.1, C6.1, C71.1, C75.1, C80.1, C84.1, C95.1, C97.1, C99.1, R22.1, R25.1, U3.1 (Vin)
- net +5V: now also R3.1
- net GND: now also R22.2, R25.2, C101.2, U9.64 (GND), U9.81 (GND); no longer C21.2, C23.2, R23.2, R24.2, R26.2, Y1.2, Y1.4
- net SD_CMD: now also U13.1 (A1); no longer U13.7 (A6)
- net SD_D0: now also U13.6 (A5); no longer U13.8 (A7)
- net SD_D1: now also U13.5 (A4); no longer U13.9 (A8)
- net SD_D2: now also U13.4 (A3); no longer U13.1 (A1)
- net USB1_DN: now also U9.69 (USB_DM_UP)
- net USB1_DP: now also U9.70 (USB_DP_UP)
- net USB1_RXN: now also U9.65 (USB_SSRXM_UP)
- net USB1_RXP: now also U9.66 (USB_SSRXP_UP)
- net USB1_TXN: now also U9.62 (USB_SSTXM_UP)
- net USB1_TXP: now also U9.63 (USB_SSTXP_UP)
- net USBH_1A_RXN: now also U9.7 (USB_SSRXM_DN0)
- net USBH_1A_RXP: now also U9.6 (USB_SSRXP_DN0)
- net USBH_1A_TXN: now also U9.9 (USB_SSTXM_DN0)
- net USBH_1A_TXP: now also U9.8 (USB_SSTXP_DN0)
- net USBH_1B_RXN: now also U9.12 (USB_SSRXP_DN2)
- net USBH_1B_RXP: now also U9.13 (USB_SSRXM_DN2)
- net USBH_1B_TXN: now also U9.14 (USB_SSTXP_DN2)
- net USBH_1B_TXP: now also U9.15 (USB_SSTXM_DN2)
- net USBH_1_DN: now also U9.3 (USB_DM_DN0)
- net USBH_1_DP: now also U9.2 (USB_DP_DN0)
- net USBH_2A_RXN: now also U9.53 (USB_SSRXP_DN1)
- net USBH_2A_RXP: now also U9.54 (USB_SSRXM_DN1)
- net USBH_2A_TXN: now also U9.55 (USB_SSTXP_DN1)
- net USBH_2A_TXP: now also U9.56 (USB_SSTXM_DN1)
- net USBH_2B_RXN: now also U9.47 (USB_SSRXP_DN3)
- net USBH_2B_RXP: now also U9.48 (USB_SSRXM_DN3)
- net USBH_2B_TXN: now also U9.49 (USB_SSTXP_DN3)
- net USBH_2B_TXP: now also U9.50 (USB_SSTXM_DN3)
- net USBH_2_DN: now also U9.59 (USB_DM_DN1)
- net USBH_2_DP: now also U9.60 (USB_DP_DN1)
- net USBH_3_DN: now also U9.18 (USB_DM_DN2)
- net USBH_3_DP: now also U9.17 (USB_DP_DN2)
- net USBH_4_DN: now also U9.44 (USB_DM_DN3)
- net USBH_4_DP: now also U9.45 (USB_DP_DN3)
- net SDC_CMD: now reaches U13.20 (B1)
- net SDC_CMD: now also J2.3 (CMD); no longer J2.1 (DAT2)
- net SDC_D3: now reaches J2.2 (DAT3/CD), U13.18 (B2)
- net at U13.14 (B6): no longer J2.3 (CMD)
- net at U13.13 (B7): no longer J2.7 (DAT0)
- net at U13.12 (B8): no longer J2.8 (DAT1)
- net at R5.1: now also U9.33 (GRSTz)
- net USBH_3V3: now reaches R24.1
- net USBH_3V3: now also C6.1, C75.1, C80.1, C84.1, C95.1, C97.1, C99.1, R26.1, U3.1 (Vin), FB7.1, U9.19 (VDD33), U9.21 (VDD33), U9.38 (VDD33), U9.4 (VDD33), U9.43 (VDD33), U9.58 (VDD33), U9.68 (VDD33), U9.72 (VDD33), U9.77 (VDD33), U9.80 (VDD33)
- net at R23.1: now also U9.78 (USB_R1); no longer R22.2
- net SDC_D0: now reaches U13.15 (B5)
- net SDC_D0: now also J2.7 (DAT0)
- net SDC_D1: now reaches U13.16 (B4)
- net SDC_D1: now also J2.8 (DAT1)
- net SDC_D2: now reaches U13.17 (B3)
- net SDC_D2: now also J2.1 (DAT2)
- net at C21.1, Y1.1: now also R2.1, U9.74 (XO)
- net at C23.1, Y1.3: now also R2.2, U9.76 (XI)
- new net: R22.1, R3.2, U9.73 (USB_VBUS)
- new net: R25.1, U9.39 (PWRON0z_BATEN0)
- new net: R24.2, U9.35 (SDA/SMBDAT)
- new net: R23.2, U9.79 (USB_R1RTN)
- new net: R26.2, U9.40 (OVERCUR0z)
- new net: C21.2, C23.2, U9.75 (VSSOSC), Y1.2, Y1.4
- no-connect marks 193 -> 167
Other:
- note added: "TODO: these go nowhere"
- note added: "disables U1/U2 states TODO: possibly control by LPC"
- note removed: "Config 4 (Flex)"
- note removed: "TODO: usb power switches"
- note removed: "These are OK, unclear why inconsistent pin numbering in symbol"
- note removed: "Unused"
- note removed: "VBUS_DET"
- note removed: "disable battery charging"
- moved on the sheet: C100, C21, C23, C74, C79, C81, C94, C96, C98, R5, R69, Y1

Commit message: motherboard: routing snapshot
Parts:
- removed C38: 0.1uF, Capacitor_SMD:C_0402_1005Metric, symbol Device:C_Small
- added H8, H9: MountingHole_Pad, footprints:WA-SMSI-M2, symbol Mechanical:MountingHole_Pad
- R1, R100, R103, R104, R105, R106, R107, R108, R109, R11, R110, R111, R12, R13, R14, R16, R18, R19, R198, R199, R2, R20, R21, R23, R24, R25, R26, R28, R29, R3, R34, R35, R36, R37, R39, R4, R40, R41, R44, R45, R46, R47, R48, R49, R5, R50, R51, R58, R6, R60, R61, R62, R63, R64, R65, R66, R67, R69, R7, R70, R71, R72, R76, R77, R79, R8, R80, R81, R82, R83, R84, R87, R9, R90, R97, R98, R99: footprint Resistor_SMD:R_0603_1608Metric -> Resistor_SMD:R_0402_1005Metric
Connections:
- net PCIE1_RXN is gone; now on net PCIE1_RX_N: U1.54 (PCIE1_RX_N)
- net PCIE1_RXP is gone; now on net PCIE1_RX_P: U1.52 (PCIE1_RX_P)
- net PCIE1_TXN is gone; now on net PCIE1_TX_N: U1.48 (PCIE1_TX_N)
- net PCIE1_TXP is gone; now on net PCIE1_TX_P: U1.46 (PCIE1_TX_P)
- net GND: now also H8.1, H9.1
Other:
- note added: "Heatsink Mount"
- note added: "TODO: imx reset"

Commit message: motherboard: routing snapshot
Parts:
- removed U3: LM3674MFX-ADJ/NOPB, Package_TO_SOT_SMD:SOT-23-5, symbol Regulator_Switching:LM3670MF
- added D3: PMEG1020EA,115, Diode_SMD:D_SOD-323, symbol Device:D_Schottky_Small_Filled
- added R27: 0, Resistor_SMD:R_0402_1005Metric, symbol Device:R_Small
- added U3: LM2830XQMFE/NOPB, Package_TO_SOT_SMD:SOT-23-5, symbol pocket-reform:LM2830XQMFE
- C13: value 12pF -> 0.1uF; footprint Capacitor_SMD:C_0603_1608Metric -> Capacitor_SMD:C_0402_1005Metric
- C17, C6: value 10uF -> 22uF
- L2: value 2.2uH -> 3.3uH
- R10: value 200k -> 10k
- R14: value 280k -> 8.25k
Connections:
- net +1V1: now also C1.1, C100.1, C101.1, C17.1, C3.1, C70.1, C71.1, C74.1, C79.1, C81.1, C94.1, C96.1, C98.1, L2.2, R14.1, U9.1 (VDD11), U9.10 (VDD11), U9.11 (VDD11), U9.16 (VDD11), U9.20 (VDD11), U9.26 (VDD11), U9.32 (VDD11), U9.37 (VDD11), U9.42 (VDD11), U9.46 (VDD11), U9.5 (VDD11), U9.51 (VDD11), U9.52 (VDD11), U9.57 (VDD11), U9.61 (VDD11), U9.67 (VDD11), U9.71 (VDD11); no longer C26.1, C28.1, C30.1, U8.23 (DVDD), U8.45 (VREG_VOUT), U8.50 (DVDD)
- net GND: now also C13.1, D3.2 (A), U3.2 (GND)
- net STANDBY_3V3: now also C13.2
- net USBH_3V3: now also R27.1
- net at R10.1, R14.2: now also U3.3 (FB); no longer C13.2
- net at L2.1: now also D3.1 (K), U3.1 (SW)
- removed net +1V2: C1.1, C100.1, C101.1, C13.1, C17.1, C3.1, C70.1, C71.1, C74.1, C79.1, C81.1, C94.1, C96.1, C98.1, L2.2, R14.1, U9.1 (VDD11), U9.10 (VDD11), U9.11 (VDD11), U9.16 (VDD11), U9.20 (VDD11), U9.26 (VDD11), U9.32 (VDD11), U9.37 (VDD11), U9.42 (VDD11), U9.46 (VDD11), U9.5 (VDD11), U9.51 (VDD11), U9.52 (VDD11), U9.57 (VDD11), U9.61 (VDD11), U9.67 (VDD11), U9.71 (VDD11)
- net 1V2_ENABLE renamed 1V1_ENABLE
- net 1V1_ENABLE: now also U3.4 (EN)
- new net: C26.1, C28.1, C30.1, U8.23 (DVDD), U8.45 (VREG_VOUT), U8.50 (DVDD)
- new net: R27.2, U3.5 (Vin)
Other:
- note added: "1A"
- note added: "1V1"
- note added: "=1.095V"
- note added: "=3.315V"
- note added: "=5.085V"
- note removed: "600mA"
- note removed: "LM3674MFX-1.2/NOPB"
- note removed: "TODO: TUSB8040 needs up to 1A, USB7002 up to 500mA"
- note removed: "TODO: decouple"
- moved on the sheet: L2, R10, R103, R111, R14, U23

Commit message: motherboard: routing snapshot
Parts:
- added R30: 100k, Resistor_SMD:R_0402_1005Metric, symbol Device:R_Small
- added R31, R32: 0, Resistor_SMD:R_0402_1005Metric, symbol Device:R_Small
- R70: value 0 -> 100k
- R83, R84: value 0 -> 22k
Connections:
- net USBH_1_CC1 is gone; now on net +5V: R83.2
- net USBH_1_CC2 is gone; now on net +5V: R84.2
- net +1V8: now also R70.2; no longer R71.2
- net +3V3: now also R30.1
- net BACKLIGHT_EN: now also U1.105 (GPIO1_IO10)
- net DISP_EN: now also R32.2
- net IMX_RESETn: now also R30.2
- net ~{DISP_RESET}: now also R31.2
- net ~{USBH_RESET}: no longer R70.2
- net at C50.1, C51.1, FB5.1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: now also R71.2
- net at U8.4 (GPIO2): now also R31.1
- net at U8.9 (GPIO7): now also R32.1
Other:
- note removed: "TODO: imx reset"
- note removed: "TODO: these go nowhere"
- moved on the sheet: R69
