File: pocket-reform-motherboard/pocket-reform-motherboard.kicad_sch (KiCad schematic)
At the start: 286 parts, among them J1 CHARGER, J10 1-2199230-6, J11 Conn_01x33, J12 2199230-5, J13 FH35C-31S-0.3HW(50), J14 USB_C_Receptacle, J15 Conn_01x02, J16 Conn_01x03, J17 Conn_01x03, J2 DM3AT-SF-PEJM5, J3 USB_C_Receptacle, J4 09452812561, J5 SYSCTL, J6 USB_INT1, J7 HDMI_D_1.4, J8 SIM_Card, J9 USB_C_Receptacle_USB2.0, SW1 SW_DIP_x01, SW2 RESET, U1 reform2-som-connector, U10 W25Q32JVSS, U11 PCF8523T, U12 AP22815, U13 TXS0108EPW, U14 SN74AVC1T45, U15 TPD4E02B04DQA, U16 TPD4E02B04DQA, U17 TPD12S521, U18 TLV320AIC3100, U19 TPD4E02B04DQA, U2 MAX1837EUT33+T, U20 TPD4E02B04DQA, U21 TPD4E02B04DQA, U22 TPD4E02B04DQA, U23 FUSB302BMPX, U3 LM2830XQMFE/NOPB, U4 TLV1117-18, U5 TPS5450DDAR, U6 TPS5450DDAR, U7 CN301, U8 RP2040, U9 TUSB8040PFP, Y1 24MHz, Y2 12MHz 18pF, Y3 32.768 kHz

Commit message: motherboard: resolve LCSC parts
Parts:
- BT1: LCSC (none) -> C238097
- C1, C101, C25, C27, C28, C29, C3, C30, C31, C32, C33, C35, C40, C41, C42, C43, C44, C45, C46, C48, C49, C50, C53, C54, C55, C57, C59, C60, C61, C62, C63, C64, C66, C68, C69, C70, C71, C72, C73, C74, C75, C76, C77, C78, C79, C80, C81, C84, C87, C94, C96: LCSC (none) -> C1525; Manufacturer Yageo -> Samsung; Manufacturer_No CC0603JPX7R9BB104 -> CL05B104KO5NNNC
- C10, C9: LCSC (none) -> C15849; Manufacturer Taiyo Yuden -> Samsung; Manufacturer_No UMK107BJ105KA-T -> CL10A105KB8NNNC
- C100, C98: LCSC (none) -> C315248; Manufacturer Yageo -> Samsung; Manufacturer_No CC0603JPX7R9BB104 -> CL05A106MP5NUNC
- C11, C12, C18, C19, C7, C8: LCSC (none) -> C1589; Manufacturer (none) -> Samsung; Manufacturer_No (none) -> CL10B103KB8NNNC
- C123, C124, C126, C83: LCSC (none) -> C385995; Manufacturer Murata -> Taiyo Yuden; Manufacturer_No GRM188R60J476ME15D -> JDK107BBJ476MA-RE
- C13, C85, C86, C88, C89, C90, C91, C92, C93: LCSC (none) -> C1525; Manufacturer (none) -> Samsung; Manufacturer_No (none) -> CL05B104KO5NNNC
- C14: LCSC (none) -> C385995; Manufacturer (none) -> Taiyo Yuden; Manufacturer_No (none) -> JDK107BBJ476MA-RE
- C15, C16: LCSC (none) -> C2999060; Manufacturer (none) -> ROQANG; Manufacturer_No (none) -> RVT0J331M0605
- C17, C6: LCSC (none) -> C86295; Manufacturer (none) -> Samsung; Manufacturer_No (none) -> CL10A226MP8NUNE
- C2, C4, C5: LCSC (none) -> C92487; Manufacturer (none) -> Samsung; Manufacturer_No (none) -> CL10A106MO8NQNC
- C20: LCSC (none) -> C15849; Manufacturer (none) -> Samsung; Manufacturer_No (none) -> CL10A105KB8NNNC
- C21, C23: LCSC (none) -> C107040
- C26, C34, C36: LCSC (none) -> C15849; Manufacturer Yageo -> Samsung; Manufacturer_No CC0603KRX5R8BB105 -> CL10A105KB8NNNC
- C37: LCSC (none) -> C100040; Manufacturer_No CC0603JPX7R9BB104 -> CC0603KRX7R9BB102
- C39, C65: LCSC (none) -> C92487; Manufacturer Murata -> Samsung; Manufacturer_No GRM188R6YA106MA73D -> CL10A106MO8NQNC
- C47: LCSC (none) -> C1525; Manufacturer Murata -> Samsung; Manufacturer_No GRM188R6YA106MA73D -> CL05B104KO5NNNC
- C51, C56, C67: LCSC (none) -> C92487; Manufacturer Yageo -> Samsung; Manufacturer_No CC0603JPX7R9BB104 -> CL10A106MO8NQNC
- C52, C58: LCSC (none) -> C1589; Manufacturer KEMET -> Samsung; Manufacturer_No C0603C103K5RAC3190 -> CL10B103KB8NNNC
- C82: LCSC (none) -> C1623; Manufacturer Taiyo Yuden -> Samsung; Manufacturer_No TMK107B7474KA-TR -> CL10B474KA8NNNC
- C95, C97, C99: LCSC (none) -> C14445; Manufacturer Yageo -> Samsung; Manufacturer_No CC0603JPX7R9BB104 -> CL05A105KP5NNNC
- D1, D23: LCSC (none) -> C72044; Manufacturer ROHM -> Everlight; Manufacturer_No SMLEN3WBC8W1 -> 19-217/R6C-AL1M2VY/3T
- D10: LCSC (none) -> C264519; Manufacturer (none) -> Everlight; Manufacturer_No (none) -> 19-337/R6GHBHC-A01/2T
- D11: value SS54? -> SS54; LCSC (none) -> C22452; Manufacturer (none) -> MDD; Manufacturer_No (none) -> SS54
- D12: LCSC (none) -> C143772
- D2, D4, D5, D6: value PMEG3050EP,115 -> PMEG4050EP,115; LCSC (none) -> C96235; Manufacturer (none) -> Nexperia; Manufacturer_No (none) -> PMEG4050EP,115
- D3: LCSC (none) -> C426863; Manufacturer (none) -> Nexperia; Manufacturer_No (none) -> PMEG1020EA,115
- D7: LCSC (none) -> C85088; Manufacturer (none) -> Nexperia; Manufacturer_No (none) -> BZX84-C5V6,215
- D8, D9: LCSC (none) -> C72044; Manufacturer (none) -> Everlight; Manufacturer_No (none) -> 19-217/R6C-AL1M2VY/3T
- FB1, FB7: LCSC (none) -> C88980; Manufacturer_No BLM18PG221SH1D -> BLM18KG221SN1D
- FB10, FB2, FB3, FB4, FB5, FB8, FB9: LCSC (none) -> C14709; Manufacturer_No BLM18KG101TN1D -> BLM18PG121SN1D
- GFX1, H1, H2, H3, H4, J14, J16, J17, J3, J4, R62, R63, R64: LCSC (none) -> DNP
- H5, H6, H7: LCSC (none) -> C2916384; Manufacturer_Name (none) -> Sinhoo; Manufacturer_Part_Number (none) -> SMTSO2020MTJ
- H8, H9: LCSC (none) -> C2916384; Manufacturer (none) -> Sinhoo; Manufacturer_No (none) -> SMTSO2020MTJ
- J1: LCSC (none) -> C278795; Manufacturer (none) -> HR(Joint Tech Elec); Manufacturer_No (none) -> A2001WR-S-09PD01
- J10: LCSC (none) -> Global Sourcing
- J11: LCSC (none) -> C597986
- J12: LCSC (none) -> C590854; Manufacturer (none) -> TE; Manufacturer_No (none) -> 1-2199230-5
- J13: LCSC (none) -> Global Sourcing; Manufacturer (none) -> TE; Manufacturer_No (none) -> 3-2328724-1
- J15: LCSC (none) -> C189893; Manufacturer (none) -> JST; Manufacturer_No (none) -> SM02B-GHS-TB(LF)(SN)
- J2: Manufacturer (none) -> Hirose; Manufacturer_No (none) -> DM3AT-SF-PEJM5
- J5: LCSC (none) -> C265332; Manufacturer (none) -> JST; Manufacturer_No (none) -> B4B-PH-K-S(LF)(SN)
- J6: LCSC (none) -> C265332
- J7: LCSC (none) -> C585444; Manufacturer (none) -> Molex; Manufacturer_No (none) -> 467650001
- J8: LCSC (none) -> C127364; Manufacturer (none) -> Molex; Manufacturer_No (none) -> 788000001
- J9: LCSC (none) -> C165948; Manufacturer (none) -> Korean Hroparts; Manufacturer_No (none) -> TYPE-C-31-M-12
- L1: LCSC (none) -> C92953; Manufacturer (none) -> Taiyo Yuden; Manufacturer_No (none) -> NRH3012T220MN
- L2: LCSC (none) -> C337905; Manufacturer (none) -> Murata; Manufacturer_No (none) -> LQH32PN3R3NN0L
- L3, L4: LCSC (none) -> C511026; Manufacturer_No (none) -> IHLP4040DZER150M11
- MK1: LCSC (none) -> C2827528; Manufacturer (none) -> STMicroelectronics; Manufacturer_No (none) -> MP23ABS1TR
- R1, R110: LCSC (none) -> C106235; Manufacturer_No RC0603FR-071KL -> RC0402FR-071KL
- R10, R15, R17, R24, R25, R26: LCSC (none) -> C60490; Manufacturer (none) -> Yageo; Manufacturer_No (none) -> RC0402FR-0710KL
- R100, R98, R99: LCSC (none) -> C144757; Manufacturer Vishay Dale -> Yageo; Manufacturer_No CRCW060347K0FKEAC -> AC0402FR-0747KL
- R103, R111, R27, R31, R32, R44, R45, R46, R49, R50, R51, R71, R9: LCSC (none) -> C242160; Manufacturer (none) -> Panasonic; Manufacturer_No (none) -> ERJ2GE0R00X
- R104, R105, R106, R107, R108, R109, R11, R12, R13, R4, R5, R67, R81: LCSC (none) -> C242160; Manufacturer Vishay Dale -> Panasonic; Manufacturer_No CRCW06030000Z0EAC -> ERJ2GE0R00X
- R14: LCSC (none) -> C852942; Manufacturer (none) -> Yageo; Manufacturer_No (none) -> RT0402BRD078K25L
- R16: LCSC (none) -> C163466; Manufacturer (none) -> Yageo; Manufacturer_No (none) -> RC0402FR-073K16L
- R18: value 5.83k -> 5.76k; LCSC (none) -> C852862; Manufacturer (none) -> Yageo; Manufacturer_No (none) -> RT0402BRD075K76L
- R19: LCSC (none) -> C203121; Manufacturer_No CR0603-FX-8873ELF -> CR0402-JW-135GLF
- R198, R199, R65, R66: LCSC (none) -> C87044; Manufacturer_No RC0603FR-1049R9L -> RC0402FR-0749R9L
- R2: LCSC (none) -> C144787; Manufacturer (none) -> Yageo; Manufacturer_No (none) -> AC0402FR-071ML
- R20: LCSC (none) -> C144057; Manufacturer Panasonic -> Yageo; Manufacturer_No ERJ-P03F1203V -> AF0402JR-07300KL
- R21: LCSC (none) -> C144787; Manufacturer Bourns -> Yageo; Manufacturer_No CR0603-FX-8873ELF -> AC0402FR-071ML
- R22: value R_Small -> 10k; LCSC (none) -> C60490; Manufacturer (none) -> Yageo
- R23: LCSC (none) -> C400642; Manufacturer (none) -> Panasonic; Manufacturer_No (none) -> ERJ2RKF9091X
- R28: LCSC (none) -> C93945; Manufacturer Bourns -> Yageo; Manufacturer_No CR0603-FX-8873ELF -> RC0402FR-07120KL
- R29, R34, R58, R60, R61: LCSC (none) -> C106235; Manufacturer (none) -> Yageo; Manufacturer_No (none) -> RC0402FR-071KL
- R3: LCSC (none) -> C26989; Manufacturer (none) -> UNI-ROYAL; Manufacturer_No (none) -> 0402WGF9092TCE
- R30, R6, R69, R7, R70, R8, R87: LCSC (none) -> C60491; Manufacturer (none) -> Yageo; Manufacturer_No (none) -> RC0402FR-07100KL
- R35: LCSC C105428 -> C106235; Manufacturer_No RC0603FR-074K7L -> RC0402FR-071KL
- R36: LCSC (none) -> C106235; Manufacturer Generic -> Yageo; Manufacturer_No GPR060310K -> RC0402FR-071KL
- R37, R39, R40, R41: LCSC (none) -> C413061; Manufacturer (none) -> Panasonic; Manufacturer_No (none) -> ERJ2RKF75R0X
- R38, R56: LCSC (none) -> C60490; Manufacturer Generic -> Yageo; Manufacturer_No GPR060310K -> RC0402FR-0710KL
- R47, R48: LCSC (none) -> C31439; Manufacturer (none) -> UNI-ROYAL; Manufacturer_No (none) -> 0402WGF274JTCE
- R57, R59: LCSC C105428 -> C105871; Manufacturer_No RC0603FR-074K7L -> RC0402FR-074K7L
- R68, R85, R96: LCSC (none) -> C60490; Manufacturer_No RC0603FR-0710KL -> RC0402FR-0710KL
- R72: LCSC (none) -> C114762; Manufacturer (none) -> Yageo; Manufacturer_No (none) -> RC0402FR-072K2L
- R75: LCSC (none) -> C60490; Manufacturer_No RC0603FR-071K5L -> RC0402FR-0710KL
- R76, R77, R79, R80, R82: LCSC (none) -> C138002; Manufacturer Vishay Dale -> Yageo; Manufacturer_No CRCW060333R0FKEAC -> RC0402FR-0733RL
- R83, R84: LCSC (none) -> C144778; Manufacturer (none) -> Yageo; Manufacturer_No (none) -> AC0402FR-0722KL
- R89, R93: LCSC (none) -> C105871; Manufacturer_No RC0603FR-074K7L -> RC0402FR-074K7L
- R90: LCSC (none) -> C413101; Manufacturer Bourns -> Panasonic; Manufacturer_No CR0603-FX-2702ELF -> ERJ2RKF2702X
- R97: LCSC (none) -> C144757; Manufacturer Vishay Dale -> Yageo; Manufacturer_No CRCW0603100KJNEAC -> AC0402FR-0747KL
- SW1: LCSC (none) -> C402914; Manufacturer Wuerth -> Dongguan Guangzhu; Manufacturer_No 418121270801 -> DSIC01LSGET
- SW2: LCSC (none) -> C318893; Manufacturer C&K -> XKB; Manufacturer_No KMR221GLFS -> TS-1185EC-C-D-B
- TR1: LCSC (none) -> C501477; Manufacturer (none) -> Heling; Manufacturer_No (none) -> MT24-S1T1
- U1: LCSC (none) -> C591654; Manufacturer (none) -> TE; Manufacturer_No (none) -> 1473149-4
- U10: LCSC (none) -> C179173; Manufacturer (none) -> Winbond; Manufacturer_No (none) -> W25Q32JVSS
- U11: LCSC (none) -> C2651516
- U12: LCSC (none) -> C2150272
- U13: LCSC (none) -> C17206
- U14: LCSC (none) -> C131978; Manufacturer_No SN74AVC1T45 -> SN74AVC1T45DBVR
- U15, U16, U19, U20, U21, U22: LCSC (none) -> C2841426; Manufacturer (none) -> Texas Instruments; Manufacturer_No (none) -> TPD4E02B04DQAR-TP
- U17: LCSC (none) -> C126920
- U18: LCSC (none) -> C478458; Manufacturer (none) -> Texas Instruments; Manufacturer_No (none) -> TLV320AIC3100
- U2: LCSC (none) -> C141779; Manufacturer (none) -> Maxim; Manufacturer_No (none) -> MAX1837EUT33+T
- U23: LCSC (none) -> C132291; Manufacturer (none) -> ON Semi; Manufacturer_No (none) -> FUSB302BMPX
- U3: LCSC (none) -> C2072452; Manufacturer (none) -> Texas Instruments; Manufacturer_No (none) -> LM2830XQMFE/NOPB
- U4: LCSC (none) -> C2862410
- U5, U6: LCSC (none) -> C114425; Manufacturer (none) -> Texas Instruments; Manufacturer_No (none) -> TPS5450DDAR
- U7: LCSC (none) -> C63355
- U8: LCSC (none) -> C2040; Manufacturer (none) -> Raspberry Pi; Manufacturer_No (none) -> RP2040
- U9: LCSC (none) -> C2872001; Manufacturer (none) -> Texas Instruments; Manufacturer_No (none) -> TUSB8040PFP
- Y1: LCSC (none) -> C91744; Manufacturer Abracon -> Seiko Epson; Manufacturer_No ABM8AIG-24.000MHz-R40-4-T -> X1E0000210264
- Y3: LCSC (none) -> C48615; Manufacturer ECS -> Seiko Epson; Manufacturer_No ECS-.327-7-34B-TR -> Q13FC1350000200
Other:
- note added: "=3.34V"
- note removed: "=3.315V"
