File: pocket-reform-motherboard/pocket-reform-motherboard.kicad_sch (KiCad schematic)
At the start: 286 parts, among them J1 CHARGER, J10 1-2199230-6, J11 Conn_01x33, J12 2199230-5, J13 FH35C-31S-0.3HW(50), J14 USB_C_Receptacle, J15 Conn_01x02, J16 Conn_01x03, J17 Conn_01x03, J2 DM3AT-SF-PEJM5, J3 USB_C_Receptacle, J4 09452812561, J5 SYSCTL, J6 USB_INT1, J7 HDMI_D_1.4, J8 SIM_Card, J9 USB_C_Receptacle_USB2.0, SW1 SW_DIP_x01, SW2 RESET, U1 reform2-som-connector, U10 W25Q32JVSS, U11 PCF8523T, U12 AP22815, U13 TXS0108EPW, U14 SN74AVC1T45, U15 TPD4E02B04DQA, U16 TPD4E02B04DQA, U17 TPD12S521, U18 TLV320AIC3100, U19 TPD4E02B04DQA, U2 MAX1837EUT33+T, U20 TPD4E02B04DQA, U21 TPD4E02B04DQA, U22 TPD4E02B04DQA, U23 FUSB302BMPX, U3 LM2830XQMFE/NOPB, U4 TLV1117-18, U5 TPS5450DDAR, U6 TPS5450DDAR, U7 CN301, U8 RP2040, U9 TUSB8040PFP, Y1 24MHz, Y2 12MHz 18pF, Y3 32.768 kHz

Commit message: motherboard: d-1 ordered version
Parts:
- added GFX2: MountingHole, footprints:pref-motherboard-badge, symbol Mechanical:MountingHole
- added R33: 0, Resistor_SMD:R_0402_1005Metric, symbol Device:R_Small
- added R42, R43: 4.7k, Resistor_SMD:R_0402_1005Metric, symbol Device:R_Small
- added TP1: TestPoint, TestPoint:TestPoint_Pad_D1.0mm, symbol Connector:TestPoint
- C123, C124, C126, C14, C83: LCSC C385995 -> C140782; Manufacturer Taiyo Yuden -> Murata; Manufacturer_No JDK107BBJ476MA-RE -> GRM188R60J476ME15D
- C15, C16: LCSC C2999060 -> C286137; Manufacturer ROQANG -> Lelon; Manufacturer_No RVT0J331M0605 -> VZT331M0JTR-0606ACS
- H5, H6, H7: LCSC C2916384 -> C2915626; Manufacturer_No 9774020243R -> SMTSO2020CTJ
- H8, H9: LCSC C2916384 -> C2915626; Manufacturer_No SMTSO2020MTJ -> SMTSO2020CTJ
- J11: LCSC C597986 -> C262220; Manufacturer Hirose -> Jushuo; Manufacturer_No FH12-33S-0.5SH(55) -> AFC07-S33FCC-00
- L1: Manufacturer Taiyo Yuden -> YJYCOIN; Manufacturer_No NRH3012T220MN -> YNR3015-150M
- L5, L6: LCSC C223122 -> C497563
- R14: LCSC C852942 -> C95598; Manufacturer Yageo -> UNI-ROYAL; Manufacturer_No RT0402BRD078K25L -> 0402WGF8251TCE
- R18: LCSC C852862 -> C25910; Manufacturer Yageo -> UNI-ROYAL; Manufacturer_No RT0402BRD075K76L -> 0402WGF5761TCE
- R19: LCSC C203121 -> C226868; Manufacturer Bourns -> Yageo; Manufacturer_No CR0402-JW-135GLF -> AC0402FR-071M3L
- R22: Manufacturer_No (none) -> RC0402FR-0710KL
- R62, R63, R64: Manufacturer_No (none) -> DNP
- U4: LCSC C2862410 -> C463601; Manufacturer Texas Instruments -> ON; Manufacturer_No TLV1117-18CDCYR -> NCV1117ST18T3G
Connections:
- net ~{M_WOWWAN} is gone; now on net RP_WOWWAN: J12.23
- net ~{M_W_DISABLE1} is gone; now on net RP_FLIGHTMODE: J12.8
- net ~{M_W_DISABLE2} is gone; now on net RP_FLIGHTMODE: J12.26
- net +1V8: now also U4.4 (VO)
- net DAC_SCL: now also R42.1
- net DAC_SDA: now also R43.1
- net GND: now also J2.P1 (SHIELD), J2.P2 (SHIELD), J2.P3 (SHIELD), J2.P4 (SHIELD), J2.SWA (DET_A), J8.P1 (SHIELD), J8.P2 (SHIELD), J8.P3 (SHIELD), J8.P4 (SHIELD), U1.111 (GND), U1.117 (GND), U1.123 (GND), U1.95 (GND), U1.99 (GND); no longer J2.10 (DET_A), J2.11 (SHIELD)
- net M2B_RST: now also TP1.1
- net SD_DET: now also J2.SWB (DET_B); no longer J2.9 (DET_B)
- net STANDBY_3V3: now also R42.2, R43.2
- net USB_SRC_EN: now also R33.2
- net at U8.40 (GPIO28_ADC2): now also R33.1
- net RP_FLIGHTMODE: now reaches U8.5 (GPIO3)
- net RP_WOWWAN: now reaches U8.8 (GPIO6)
- no-connect marks 167 -> 185
Other:
- note added: "D-2 TODO: - change HDMI connector to LCSC part - change USB3 connector to LCSC part"
- note added: "Needs inrush limiter and UVLO on charger board!"
- note removed: "Needs inrush limiter on charger board!"
- note removed: "TODO: R27 needed?"
- note removed: "TODO: SATA config jumper for LS1028A"
- note removed: "TODO: confirm"
- note removed: "TODO: confirm pinout!"
- moved on the sheet: R30

Commit message: motherboard: add some notes
Connections:
- no-connect marks 185 -> 189
Other:
- note added: "DCDC_EN"
- note added: "MAX 24V"
- note added: "MAX 36V"
- note added: "TODO unconnected"
- note added: "TODO: could be 5V TODO: caps"
- note added: "TODO: replace with SMD part"
- note added: "TODO: reset level 1.8!"
- note added: "TODO: wrong connector"
- note added: "TODO: wrong! must be 3V3!!!"
- note added: "XRES"
- note added: "actually 12401548E412A"
- note added: "wrong part (1473149-4)! the correct one is 1473149-1!"
Changed lines of the file:
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@@
   (no_connect (at 756.92 598.17))
   (no_connect (at 756.92 572.77))
+  (no_connect (at 471.17 256.54))
+  (no_connect (at 471.17 261.62))
+  (no_connect (at 471.17 264.16))
+  (no_connect (at 471.17 266.7))
   (no_connect (at 759.46 389.89))
   (no_connect (at 580.39 254))
@@
     (effects (font (size 2.54 2.54)) (justify left bottom))
   )
+  (text "MAX 24V" (at 168.91 99.06 0)
+    (effects (font (size 1.27 1.27)) (justify left bottom))
+  )
   (text "Backlight is digitally controlled" (at 801.37 179.07 0)
     (effects (font (size 1.27 1.27)) (justify left bottom))
@@
     (effects (font (size 1.27 1.27)) (justify left bottom))
   )
+  (text "TODO: wrong! must be 3V3!!!" (at 453.39 158.115 0)
+    (effects (font (size 1.27 1.27)) (justify left bottom))
+  )
   (text "PETp3" (at 728.98 556.26 0)
     (effects (font (size 1.27 1.27)) (justify left bottom))
@@
     (effects (font (size 1.27 1.27)) (justify right bottom))
   )
+  (text "TODO: reset level 1.8!" (at 734.06 202.565 0)
+    (effects (font (size 1.27 1.27)) (justify left bottom))
+  )
   (text "D-2 TODO:\n\n- change HDMI connector to LCSC part\n- change USB3 connector to LCSC part\n"
     (at 38.1 169.545 0)
@@
     (effects (font (size 1.27 1.27)) (justify left bottom))
   )
+  (text "MAX 36V" (at 169.545 202.565 0)
+    (effects (font (size 1.27 1.27)) (justify left bottom))
+  )
   (text "PERp2" (at 728.98 563.88 0)
     (effects (font (size 1.27 1.27)) (justify left bottom))
@@
     (effects (font (size 1.27 1.27)) (justify left bottom))
   )
+  (text "TODO: replace with SMD part" (at 918.21 166.37 0)
+    (effects (font (size 1.27 1.27)) (justify left bottom))
+  )
   (text "Serial Ports" (at 728.98 41.91 0)
     (effects (font (size 2.54 2.54)) (justify left bottom))
@@
     (effects (font (size 1.27 1.27)) (justify left bottom))
   )
+  (text "actually 12401548E412A " (at 922.02 54.61 0)
+    (effects (font (size 1.27 1.27)) (justify left bottom))
+  )
   (text "TODO: CLKGEN for imx8mq?" (at 641.35 434.34 0)
     (effects (font (size 1.27 1.27)) (justify left bottom))
@@
     (effects (font (size 1.27 1.27)) (justify left bottom))
   )
+  (text "wrong part (1473149-4)! the correct one is 1473149-1!"
+    (at 186.055 354.33 0)
+    (effects (font (size 1.27 1.27)) (justify left bottom))
+  )
   (text "MicroSD Slot" (at 928.37 463.55 0)
     (effects (font (size 2.54 2.54)) (justify left bottom))
@@
     (effects (font (size 1.27 1.27)) (justify left bottom))
   )
+  (text "TODO: could be 5V\nTODO: caps" (at 771.525 142.875 0)
+    (effects (font (size 1.27 1.27)) (justify left bottom))
+  )
   (text "=1.095V" (at 240.665 262.89 0)
     (effects (font (size 1.27 1.27)) (justify left bottom))
@@
     (effects (font (size 1.27 1.27)) (justify left bottom))
   )
+  (text "DCDC_EN" (at 791.845 222.885 0)
+    (effects (font (size 1.27 1.27)) (justify left bottom))
+  )
   (text "250mA" (at 198.12 127 0)
     (effects (font (size 1.27 1.27)) (justify left bottom))
@@
     (effects (font (size 2.54 2.54)) (justify left bottom))
   )
+  (text "TODO unconnected" (at 260.985 579.12 0)
+    (effects (font (size 1.27 1.27)) (justify left bottom))
+  )
   (text "Port\nProtection" (at 965.2 359.41 0)
     (effects (font (size 1.27 1.27)) (justify left bottom))
   )
+  (text "TODO: replace with SMD part" (at 920.115 58.42 0)
+    (effects (font (size 1.27 1.27)) (justify left bottom))
+  )
   (text "TX caps are on the SoM" (at 688.34 417.83 0)
     (effects (font (size 1.27 1.27)) (justify left bottom))
   )
+  (text "TODO: wrong connector" (at 1063.625 686.435 0)
+    (effects (font (size 1.27 1.27)) (justify left bottom))
+  )
   (text "NRH3012T220MN" (at 215.9 102.87 0)
     (effects (font (size 1.27 1.27)) (justify left bottom))
@@
     (effects (font (size 1.27 1.27)) (justify left bottom))
   )
+  (text "MAX 36V" (at 169.545 157.48 0)
+    (effects (font (size 1.27 1.27)) (justify left bottom))
+  )
   (text "PERn1" (at 728.98 576.58 0)
     (effects (font (size 1.27 1.27)) (justify left bottom))
@@
     (effects (font (size 1.27 1.27)) (justify left bottom))
   )
+  (text "XRES" (at 791.845 207.01 0)
+    (effects (font (size 1.27 1.27)) (justify left bottom))
+  )
   (text "TODO" (at 741.68 210.82 0)
     (effects (font (size 1.27 1.27)) (justify left bottom))
@@
     (pin "7")
     (pin "8")
-    (pin "SWB")
     (pin "P1")
     (pin "P2")
@@
     (pin "P4")
     (pin "SWA")
+    (pin "SWB")
   )
   (symbol (lib_id "Connector:Conn_01x09_Male") (at 46.99 87.63 0) (unit 1)

Commit message: d-2 pcbs TODO
Connections:
- net USB1_RXN: now also U9.62 (USB_SSTXM_UP); no longer U9.65 (USB_SSRXM_UP)
- net USB1_RXP: now also U9.63 (USB_SSTXP_UP); no longer U9.66 (USB_SSRXP_UP)
- net USB1_TXN: now also U9.65 (USB_SSRXM_UP); no longer U9.62 (USB_SSTXM_UP)
- net USB1_TXP: now also U9.66 (USB_SSRXP_UP); no longer U9.63 (USB_SSTXP_UP)
Other:
- note added: "I2C control bus"
- note added: "NOTE: TX/RX were swapped in D-1"
- note added: "TODO: footprint needs more GND EP solder paste! this caused a failure on 1/3 boards"
- note added: "TODO: these should not be connected"
- note added: "TODO: these shouldn't go to STANDBY_3V3 because of V leak into som?"
- note added: "TODO: this R is too large for imx8mplus! changed to 10k on board"
- note removed: "Needs inrush limiter and UVLO on charger board!"
- moved on the sheet: D2, J1

Commit message: WIP: work on mb schematic
Parts:
- removed C20: 1uF, Capacitor_SMD:C_0603_1608Metric, symbol Device:C_Small
- removed C68, C69: 0.1uF, Capacitor_SMD:C_0402_1005Metric, symbol Device:C_Small
- removed D7: BZX84-C5V6,215, Diode_SMD:D_SOD-323, symbol reform2-batterypack-upstream-rescue:D_Zener_Small_ALT-Device
- removed MK1: MP23ABS1TR, footprints:MIC_MP23ABS1TR, symbol MP23ABS1TR:MP23ABS1TR
- removed R19: 1.3M, Resistor_SMD:R_0402_1005Metric, symbol Device:R_Small
- removed R20: 300k, Resistor_SMD:R_0402_1005Metric, symbol Device:R_Small
- removed R21: 1M, Resistor_SMD:R_0402_1005Metric, symbol Device:R_Small
- removed R28: 120k, Resistor_SMD:R_0402_1005Metric, symbol Device:R_Small
- removed R72: 2k2, Resistor_SMD:R_0402_1005Metric, symbol Device:R_Small
- removed U7: CN301, Package_TO_SOT_SMD:SOT-23-5, symbol reform2-batterypack:CN301
- added J18: Conn_01x05_Socket, symbol Connector:Conn_01x05_Socket
- BT1: value V364 -> V364 DNP
- J15: footprint Connector_JST:JST_GH_SM02B-GHS-TB_1x02-1MP_P1.25mm_Horizontal -> Connector_Molex:Molex_PicoBlade_53261-0271_1x02-1MP_P1.25mm_Horizontal; LCSC C189893 -> (none); Manufacturer JST -> Molex; Manufacturer_No SM02B-GHS-TB(LF)(SN) -> 53261-7002
- R30: value 100k -> 10k; Manufacturer_No RC0402FR-07100KL -> (none)
- U1: LCSC C591654 -> (none); Manufacturer_No 1473149-4 -> 1473149-1
Connections:
- net +3V3: now also R42.2, R43.2
- net +5V: no longer C40.1, U8.48 (USB_VDD)
- net STANDBY_3V3: now also C40.1, U8.48 (USB_VDD); no longer R42.2, R43.2
- no-connect marks 189 -> 190
Other:
- note added: "1473149-4 is incompatible! the correct one is 1473149-1! (or 1717254-1)"
- note added: "1Gb Ethernet"
- note added: "TODO switch/jumper"
- note added: "TODO: connector for headphone/mic"
- note removed: "Input UVLO"
- note removed: "MEMS microphone"
- note removed: "Optional 1Gb Ethernet"
- note removed: "TODO"
- note removed: "TODO: these shouldn't go to STANDBY_3V3 because of V leak into som?"
- note removed: "TODO: this R is too large for imx8mplus! changed to 10k on board"
- note removed: "TODO: wrong connector"
- note removed: "TODO: wrong! must be 3V3!!!"
- note removed: "wrong part (1473149-4)! the correct one is 1473149-1!"
- moved on the sheet: C40

Commit message: WIP: motherboard:  move things around
Parts:
- J5, J6: footprint Connector_JST:JST_PH_S4B-PH-SM4-TB_1x04-1MP_P2.00mm_Horizontal -> Connector_JST:JST_SH_SM04B-SRSS-TB_1x04-1MP_P1.00mm_Horizontal; LCSC C265332 -> (none); Manufacturer_No B4B-PH-K-S(LF)(SN) -> (none)
Changed lines of the file:
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@@
       (effects (font (size 1.27 1.27)))
     )
-    (property "Footprint" "Connector_JST:JST_PH_S4B-PH-SM4-TB_1x04-1MP_P2.00mm_Horizontal" (at 438.15 614.68 0)
+    (property "Footprint" "Connector_JST:JST_SH_SM04B-SRSS-TB_1x04-1MP_P1.00mm_Horizontal" (at 438.15 614.68 0)
       (effects (font (size 1.27 1.27)) hide)
     )
@@
       (effects (font (size 1.27 1.27)) hide)
     )
-    (property "Manufacturer_No" "B4B-PH-K-S(LF)(SN)" (at 438.15 614.68 0)
+    (property "Manufacturer_No" "" (at 438.15 614.68 0)
       (effects (font (size 1.27 1.27)) hide)
     )
@@
       (effects (font (size 1.27 1.27)) hide)
     )
-    (property "LCSC" "C265332" (at 438.15 614.68 0)
+    (property "LCSC" "" (at 438.15 614.68 0)
       (effects (font (size 1.27 1.27)) hide)
     )
@@
       (effects (font (size 1.27 1.27)))
     )
-    (property "Footprint" "Connector_JST:JST_PH_S4B-PH-SM4-TB_1x04-1MP_P2.00mm_Horizontal" (at 405.13 614.68 0)
+    (property "Footprint" "Connector_JST:JST_SH_SM04B-SRSS-TB_1x04-1MP_P1.00mm_Horizontal" (at 405.13 614.68 0)
       (effects (font (size 1.27 1.27)) hide)
     )
@@
       (effects (font (size 1.27 1.27)) hide)
     )
-    (property "LCSC" "C265332" (at 405.13 614.68 0)
+    (property "LCSC" "" (at 405.13 614.68 0)
       (effects (font (size 1.27 1.27)) hide)
     )
@@
       (effects (font (size 1.27 1.27)) hide)
     )
-    (property "Manufacturer_No" "B4B-PH-K-S(LF)(SN)" (at 405.13 614.68 0)
-      (effects (font (size 1.27 1.27)) hide)
-    )
+    (property "Manufacturer_No" "" (at 405.13 614.68 0)
+      (effects (font (size 1.27 1.27)) hide)
+    )

Commit message: WIP: mb: more shuffling
Parts:
- removed BT1: V364 DNP, Battery:BatteryHolder_Keystone_2998_1x6.8mm, symbol Device:Battery_Cell
- removed C41: 0.1uF, Capacitor_SMD:C_0402_1005Metric, symbol Device:C_Small
- removed J16, J17: Conn_01x03, Connector_PinHeader_2.54mm:PinHeader_1x03_P2.54mm_Vertical, symbol Connector_Generic:Conn_01x03
- added C20: 0.1uF, Capacitor_SMD:C_0402_1005Metric, symbol Device:C_Small
- added J16: SAMTEC_TSM-106-02-X-SH-A, footprints:SAMTEC_TSM-106-02-X-SH-A, symbol Connector_Generic:Conn_01x06
- added R19: 0, Resistor_SMD:R_0402_1005Metric, symbol Device:R_Small
- added R20: 10k, Resistor_SMD:R_0402_1005Metric, symbol Device:R_Small
- added U7: 74LVC1G34, Package_TO_SOT_SMD:SOT-23-5, symbol 74xGxx:74LVC1G34
- J14, J3: footprint Connector_USB:USB_C_Receptacle_Amphenol_12401548E4-2A_CircularHoles -> footprints:MOLEX_105450-0101; LCSC DNP -> C134092
Connections:
- net +1V8: now also J13.1 (Pin_1), C20.1, U7.5 (VCC); no longer J13.31 (Pin_31)
- net +3V3: now also J13.28 (Pin_28), J13.29 (Pin_29), J13.30 (Pin_30), J13.31 (Pin_31), J13.5 (Pin_5), J13.6 (Pin_6); no longer J13.1 (Pin_1), J13.2 (Pin_2), J13.26 (Pin_26), J13.27 (Pin_27), J13.3 (Pin_3), J13.4 (Pin_4)
- net BACKLIGHT_EN: now also J13.26 (Pin_26); no longer J13.6 (Pin_6)
- net DISP_EN: now also J13.2 (Pin_2); no longer J13.30 (Pin_30)
- net DISP_TE: now also J13.7 (Pin_7); no longer J13.25 (Pin_25)
- net DSI_CLK_N: now also J13.17 (Pin_17); no longer J13.15 (Pin_15)
- net DSI_D0_N: now also J13.20 (Pin_20); no longer J13.12 (Pin_12)
- net DSI_D0_P: now also J13.19 (Pin_19); no longer J13.13 (Pin_13)
- net DSI_D1_N: now also J13.14 (Pin_14); no longer J13.18 (Pin_18)
- net DSI_D1_P: now also J13.13 (Pin_13); no longer J13.19 (Pin_19)
- net DSI_D2_N: now also J13.11 (Pin_11); no longer J13.21 (Pin_21)
- net DSI_D2_P: now also J13.10 (Pin_10); no longer J13.22 (Pin_22)
- net DSI_D3_N: now also J13.23 (Pin_23); no longer J13.9 (Pin_9)
- net DSI_D3_P: now also J13.22 (Pin_22); no longer J13.10 (Pin_10)
- net GND: now also J13.12 (Pin_12), J13.15 (Pin_15), J13.18 (Pin_18), J13.21 (Pin_21), J13.24 (Pin_24), J13.27 (Pin_27), J13.3 (Pin_3), J13.4 (Pin_4), J13.9 (Pin_9), J18.1 (Pin_1), C20.2, J16.1 (Pin_1), J16.4 (Pin_4), R20.2, U7.3 (GND); no longer J13.11 (Pin_11), J13.14 (Pin_14), J13.17 (Pin_17), J13.20 (Pin_20), J13.23 (Pin_23), J13.28 (Pin_28), J13.29 (Pin_29), J13.5 (Pin_5), J13.8 (Pin_8)
- net IMX_UART1_RX: now also J16.5 (Pin_5)
- net IMX_UART1_TX: now also J16.6 (Pin_6)
- net IMX_UART2_RX: now also J16.2 (Pin_2)
- net IMX_UART2_TX: now also J16.3 (Pin_3)
- net STANDBY_3V3: now also R19.2
- net ~{DISP_RESET}: now also R20.1, U7.2; no longer J13.24 (Pin_24)
- net at U18.12 (MICBIAS): now also J18.3 (Pin_3)
- net at U18.14 (MIC1RP): now also J18.2 (Pin_2)
- net at U18.27 (HPL): now also J18.4 (Pin_4)
- net at U18.30 (HPR): now also J18.5 (Pin_5)
- net at U11.3 (VBAT): now also R19.1
- net ~{M_PWROFF} renamed MODEM_PWROFFn
- new net ~{DISP_RESET_1V8}: J13.8 (Pin_8), U7.4
- no-connect marks 190 -> 187
Other:
- note added: "1.25mm pitch Molex Picoblade"
- note added: "Flipped vertically vs D-1"
- note added: "TE"
- note added: "TE 3-2328724-1"
- note added: "TODO: PWROFF!"
- note added: "TODO: connect shield pins to GND"
- note added: "TODO: connector for headphone/mic TODO: review datasheet"
- note removed: "1.25mm pitch Molex Picoblade JST GH?"
- note removed: "Powered by coin cell when batteries removed"
- note removed: "TE 3-2328724-1 requested at snapeda"
- note removed: "TODO: connector for headphone/mic"
- moved on the sheet: J18

Commit message: motherboard schematics basically done
Parts:
- removed H6: NGFF-Mount1, footprints:WA-SMSI-M2, symbol Mechanical:MountingHole_Pad
- removed TP1: TestPoint, TestPoint:TestPoint_Pad_D1.0mm, symbol Connector:TestPoint
- added C102, C103: 47uF, Capacitor_SMD:C_0402_1005Metric, symbol Device:C_Small
- added C104, C68, C69: 0.1uF, Capacitor_SMD:C_0402_1005Metric, symbol Device:C_Small
- added C105: 10uF, Capacitor_SMD:C_0603_1608Metric, symbol Device:C_Small
- added C41: 1uF, Capacitor_SMD:C_0603_1608Metric, symbol Device:C_Small
- added FB6: 100@100MHz 3A, Inductor_SMD:L_0603_1608Metric, symbol pocket-reform-motherboard-rescue:Ferrite_Bead_Small-Device
- added J17, J19: Conn_01x03_Pin, Connector_PinHeader_2.00mm:PinHeader_1x03_P2.00mm_Vertical_SMD_Pin1Left, symbol Connector:Conn_01x03_Pin
- added J20: QWIIC, Connector_JST:JST_SH_SM04B-SRSS-TB_1x04-1MP_P1.00mm_Horizontal, symbol Connector:Conn_01x04_Pin
- added R21, R55, R74, R78: DNP, Resistor_SMD:R_0402_1005Metric, symbol Device:R_Small
- added R28, R52, R72: 10k, Resistor_SMD:R_0402_1005Metric, symbol Device:R_Small
- added R53, R54: 0, Resistor_SMD:R_0402_1005Metric, symbol Device:R_Small
- added R73: 47k, Resistor_SMD:R_0402_1005Metric, symbol Device:R_Small
- added U24: TXS0108EPW, Package_SO:TSSOP-20_4.4x6.5mm_P0.65mm, symbol Logic_LevelTranslator:TXS0108EPW
- J15: value Conn_01x02 -> CONN_SPK
- J18: value Conn_01x05_Socket -> CONN_HEAD; footprint (none) -> Connector_JST:JST_SH_SM05B-SRSS-TB_1x05-1MP_P1.00mm_Horizontal
- R63: value DNP -> 47k; LCSC DNP -> C242160; Manufacturer (none) -> Panasonic; Manufacturer_No DNP -> ERJ2GE0R00X
- R64: value DNP -> 2.2k; LCSC DNP -> C242160; Manufacturer (none) -> Panasonic; Manufacturer_No DNP -> ERJ2GE0R00X
- R65, R66: value 49.9 -> 0; Checked y -> (none); Distributor Mouser -> (none); LCSC C87044 -> C242160; Manufacturer Yageo -> Panasonic; Manufacturer_No RC0402FR-0749R9L -> ERJ2GE0R00X
Connections:
- net +1V8: now also C41.1, R53.1
- net +3V3: now also FB6.1, R54.2; no longer J13.28 (Pin_28), J13.29 (Pin_29), J13.30 (Pin_30), J13.31 (Pin_31), J13.5 (Pin_5), J13.6 (Pin_6)
- net GND: now also J13.S1 (Pin_32), J13.S2 (Pin_33), J18.5 (Pin_5), J4.3, J4.8, J4.SH, C105.2, C41.2, C68.2, C69.2, J20.1 (Pin_1), R73.2, U24.11 (GND); no longer J18.1 (Pin_1), R65.1, R66.1
- net MODEM_PWROFFn: now also U8.29 (GPIO18)
- net PCIE2_CLK_N: no longer J12.53, R65.2
- net PCIE2_CLK_P: no longer J12.55, R66.2
- net PCIE2_RESETn: no longer J12.50
- net PCIE2_RX_N: no longer J12.47
- net PCIE2_RX_P: no longer J12.49
- net PCIE2_TX_N: no longer J12.41
- net PCIE2_TX_P: no longer J12.43
- net RP_FLIGHTMODE: now also R65.2, R66.2; no longer J12.26, J12.8
- net RP_SCL0: now also J20.4 (Pin_4)
- net RP_SDA0: now also J20.3 (Pin_3)
- net RUD+: now also J19.2 (Pin_2); no longer J9.A6 (D+), J9.B6 (D+), R63.1
- net RUD-: now also J17.2 (Pin_2); no longer J9.A7 (D-), J9.B7 (D-), R64.1
- net STANDBY_3V3: now also J20.2 (Pin_2)
- net USB2_DN: now also J17.3 (Pin_3); no longer R64.2
- net USB2_DP: now also J19.3 (Pin_3); no longer R63.2
- net USB2_RXN: no longer J12.35
- net USB2_RXP: no longer J12.37
- net USB2_TXN: no longer J12.29
- net USB2_TXP: no longer J12.31
- net VCC: now also R72.1
- net ~{DISP_RESET_1V8}: now also R73.1
- net ~{STANDBY_SHDN}: now also R72.2
- net MODEM_3V3: now reaches C123.1, C52.1, C53.1, C54.1, C55.1, C83.1, FB3.2, J12.2, J12.4, J12.70, J12.72, J12.74, R1.1
- net at U1.180 (SAI3_MCLK/PWM4): now also R74.2
- net PHONE_RXFS_3V3: now reaches U1.190 (SAI3_TXFS)
- net PHONE_RXFS_3V3: now also R55.1
- net PHONE_CLK_3V3: now reaches U1.192 (SAI3_TXC)
- net PHONE_CLK_3V3: now also U24.20 (B1)
- net PHONE_DOUT_3V3: now reaches U1.194 (SAI3_RXD)
- net PHONE_DOUT_3V3: now also U24.17 (B3)
- net PHONE_DIN_3V3: now reaches U1.196 (SAI3_TXD)
- net PHONE_DIN_3V3: now also U24.18 (B2)
- net PHONE_TXFS_3V3: now reaches U1.198 (SAI3_RXFS)
- net PHONE_TXFS_3V3: now also R21.1
- net HEAD_MIC: now reaches U18.11 (VOL/MICDET)
- net HEAD_MIC: now also J18.2 (Pin_2), R64.1, C104.2
- net at U18.12 (MICBIAS): now also R64.2; no longer J18.3 (Pin_3)
- net at U18.14 (MIC1RP): now also C104.1; no longer J18.2 (Pin_2)
- net AUD_3V3: now reaches C50.1, C51.1, FB5.1, R71.2, U18.17 (AVDD), U18.28 (HPVDD)
- net AUD_3V3: now also R63.2
- net at U18.27 (HPL): now also C103.1; no longer J18.4 (Pin_4)
- net at U18.30 (HPR): now also C102.1; no longer J18.5 (Pin_5)
- net MODEM_RESET_3V3: now reaches U8.31 (GPIO20)
- net MODEM_RESET_3V3: now also U24.15 (B5)
- net PHONE_DPR_3V3: now reaches U8.39 (GPIO27_ADC1)
- net PHONE_DPR_3V3: now also U24.13 (B7)
- net BACKLIGHT_PWM: no longer names the net of U1.164 (SPDIF_RX/PWM2)
- net BACKLIGHT_PWM: now also R78.2
- net M2B_RST renamed MODEM_RESET
- net MODEM_RESET: now also U24.6 (A5)
- net M_DPR renamed PHONE_DPR
- net PHONE_DPR: now also U24.8 (A7)
- net M_I2S_CLK renamed PHONE_CLK
- net PHONE_CLK: now also U24.1 (A1)
- net M_I2S_RX renamed PHONE_DIN
- net PHONE_DIN: now also U24.3 (A2)
- net M_I2S_TX renamed PHONE_DOUT
- net PHONE_DOUT: now also U24.4 (A3)
- net M_I2S_WA renamed PHONE_SYNC
- net PHONE_SYNC: now also U24.5 (A4)
- net RP_WOWWAN renamed WOWWAN
- net WOWWAN: now also R28.2, U24.7 (A6); no longer U8.8 (GPIO6)
- new net: C68.1, R28.1, R52.1, R53.2, U24.2 (VCCA)
- new net: J18.1 (Pin_1), R63.1
- new net: R52.2, U24.10 (OE)
- new net: C69.1, R54.1, U24.19 (VCCB)
- new net: C105.1, FB6.2, J13.28 (Pin_28), J13.29 (Pin_29), J13.30 (Pin_30), J13.31 (Pin_31), J13.5 (Pin_5), J13.6 (Pin_6)
- new net HEAD_HPL: C103.2, J18.3 (Pin_3)
- new net HEAD_HPR: C102.2, J18.4 (Pin_4)
- new net PHONE_SYNC_3V3: R21.2, R55.2, U24.16 (B4)
- new net WOWWAN_3V3: U24.14 (B6), U8.8 (GPIO6)
- new net XUD+: J19.1 (Pin_1), J9.A6 (D+), J9.B6 (D+)
- new net XUD-: J17.1 (Pin_1), J9.A7 (D-), J9.B7 (D-)
- new net ~{M_W_DISABLE1}: J12.8, R65.1
- new net ~{M_W_DISABLE2}: J12.26, R66.1
- no-connect marks 187 -> 188
Other:
- note added: "1V8"
- note added: "1V8 -> 3V3"
- note added: "1V8 OD"
- note added: "1V8/3V3"
- note added: "3V3"
- note added: "Phone Level Shifter"
- note added: "Qwiic I2C Interface"
- note added: "RP2040 has 3.3V IO"
- note added: "This pair of jumpers connects RP2040 (SYSCON) to either the SOC or the J9 USB port."
- note added: "To headphone PCB"
- note added: "alt: USB7200"
- note added: "disables U1/U2 states NOTE: possibly control by LPC"
- note removed: "D-2 TODO: - change HDMI connector to LCSC part - change USB3 connector to LCSC part"
- note removed: "TODO switch/jumper"
- note removed: "TODO unconnected"
- note removed: "TODO: AC caps on USB3/PCIe? RX/TX correct?"
- note removed: "TODO: CLKGEN for imx8mq?"
- note removed: "TODO: PWROFF!"
- note removed: "TODO: Shield?"
- note removed: "TODO: connect shield pins to GND"
- note removed: "TODO: connector for headphone/mic TODO: review datasheet"
- note removed: "TODO: could be 5V TODO: caps"
- note removed: "TODO: footprint needs more GND EP solder paste! this caused a failure on 1/3 boards"
- note removed: "TODO: replace with SMD part"
- note removed: "TODO: reset level 1.8!"
- note removed: "TODO: these should not be connected"
- note removed: "TODO: voltages!"
- note removed: "TODO: we could supply 5V on VCONN"
- note removed: "actually 12401548E412A"
- note removed: "disables U1/U2 states TODO: possibly control by LPC"
- note removed: "https://www.microchipdirect.com/product/USB7002T-I/KDXVAO?productLoaded=true"
- note removed: "works only with NXP: optional internal USB connection RP/IMX"
- moved on the sheet: C2, H7, J18, R11
