File: pocket-reform-motherboard/pocket-reform-motherboard.kicad_sch (KiCad schematic)
At the start: 301 parts, among them J1 CHARGER, J10 1-2199230-6, J11 Conn_01x33, J12 2199230-5, J13 FH35C-31S-0.3HW(50), J14 USB_C_Receptacle, J15 CONN_SPK, J16 SAMTEC_TSM-106-02-X-SH-A, J18 CONN_HEAD, J2 DM3AT-SF-PEJM5, J20 QWIIC, J21 USBSEL, J3 USB_C_Receptacle, J4 09452812561, J5 SYSCTL, J6 USB_INT1, J7 HDMI_D_1.4, J8 SIM_Card, J9 USB_C_Receptacle_USB2.0, SW1 SW_DIP_x01, SW2 RESET, U1 reform2-som-connector, U10 W25Q32JVSS, U11 PCF8523T, U12 AP22815, U13 TXS0108EPW, U14 SN74AVC1T45, U15 TPD4E02B04DQA, U16 TPD4E02B04DQA, U17 TPD12S521, U18 TLV320AIC3100, U19 TPD4E02B04DQA, U2 MAX1837EUT33+T, U20 TPD4E02B04DQA, U21 TPD4E02B04DQA, U22 TPD4E02B04DQA, U23 FUSB302BMPX, U24 TXS0108EPW, U3 LM2830XQMFE/NOPB, U4 TLV1117-18, U5 TPS5450DDAR, U6 TPS5450DDAR, U7 74LVC1G34, U8 RP2040, U9 TUSB8040PFP, Y1 24MHz, Y2 12MHz 18pF, Y3 32.768 kHz

Commit message: motherboard: D-3 production snapshot
Parts:
- C102, C103: footprint Capacitor_SMD:C_0402_1005Metric -> Capacitor_SMD:C_0805_2012Metric; Checked y -> (none); LCSC C1525 -> (none); Manufacturer_No CL05B104KO5NNNC -> (none)
Changed lines of the file:
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@@
       (effects (font (size 1.27 1.27)) (justify left))
     )
-    (property "Footprint" "Capacitor_SMD:C_0402_1005Metric" (at 1007.11 706.12 0)
+    (property "Footprint" "Capacitor_SMD:C_0805_2012Metric" (at 1007.11 706.12 0)
       (effects (font (size 1.27 1.27)) hide)
     )
@@
       (effects (font (size 1.27 1.27)) hide)
     )
-    (property "Manufacturer_No" "CL05B104KO5NNNC" (at 1007.11 706.12 0)
-      (effects (font (size 1.27 1.27)) hide)
-    )
-    (property "Checked" "y" (at 1007.11 706.12 0)
+    (property "Manufacturer_No" "" (at 1007.11 706.12 0)
+      (effects (font (size 1.27 1.27)) hide)
+    )
+    (property "Checked" "" (at 1007.11 706.12 0)
       (effects (font (size 1.27 1.27)) hide)
     )
@@
       (effects (font (size 1.27 1.27)) hide)
     )
-    (property "LCSC" "C1525" (at 1007.11 706.12 0)
+    (property "LCSC" "" (at 1007.11 706.12 0)
       (effects (font (size 1.27 1.27)) hide)
     )
@@
       (effects (font (size 1.27 1.27)) (justify left))
     )
-    (property "Footprint" "Capacitor_SMD:C_0402_1005Metric" (at 1002.03 703.58 0)
+    (property "Footprint" "Capacitor_SMD:C_0805_2012Metric" (at 1002.03 703.58 0)
       (effects (font (size 1.27 1.27)) hide)
     )
@@
       (effects (font (size 1.27 1.27)) hide)
     )
-    (property "Manufacturer_No" "CL05B104KO5NNNC" (at 1002.03 703.58 0)
-      (effects (font (size 1.27 1.27)) hide)
-    )
-    (property "Checked" "y" (at 1002.03 703.58 0)
+    (property "Manufacturer_No" "" (at 1002.03 703.58 0)
+      (effects (font (size 1.27 1.27)) hide)
+    )
+    (property "Checked" "" (at 1002.03 703.58 0)
       (effects (font (size 1.27 1.27)) hide)
     )
@@
       (effects (font (size 1.27 1.27)) hide)
     )
-    (property "LCSC" "C1525" (at 1002.03 703.58 0)
-      (effects (font (size 1.27 1.27)) hide)
-    )
+    (property "LCSC" "" (at 1002.03 703.58 0)
+      (effects (font (size 1.27 1.27)) hide)
+    )

Commit message: mb: snapshot before TUSB8041 change
Parts:
- added R86: 0, Resistor_SMD:R_0402_1005Metric, symbol Device:R_Small
- added R88: DNP, Resistor_SMD:R_0402_1005Metric, symbol Device:R_Small
- C10, C104, C123, C124, C126, C20, C21, C23, C39, C46, C47, C48, C49, C50, C51, C52, C53, C54, C55, C56, C57, C58, C59, C60, C61, C62, C63, C64, C65, C66, C67, C68, C69, C72, C73, C76, C77, C78, C82, C83, C87, C9, D1, D23, FB1, FB10, FB2, FB3, FB4, FB5, FB6, FB7, FB8, FB9, J10, J11, L5, L6, R1, R100, R104, R105, R106, R107, R108, R109, R11, R110, R12, R13, R19, R198, R199, R28, R4, R5, R52, R53, R54, R67, R68, R75, R76, R77, R79, R80, R81, R82, R85, R89, R90, R93, R96, R97, R98, R99, U11, U13, U14, U17, U24, U4, Y1, Y3: Checked y -> (none); Distributor Mouser -> (none)
- C102, C103: Distributor Mouser -> (none); Manufacturer Samsung -> Taiyo Yuden; Manufacturer_No (none) -> JMK212BBJ476MG-T
- D12: Distributor Mouser -> (none)
- H5, H7: Checked y -> (none); Distributor None -> (none); Manufacturer_Name Sinhoo -> (none); Manufacturer_Part_Number SMTSO2020MTJ -> (none)
- J12: Comment 2199230-5 -> (none); EU_RoHS_Compliance Compliant -> (none)
- J14, J3: Manufacturer (none) -> Molex; Manufacturer_No (none) -> 105450-0101
- J16: Manufacturer (none) -> Samtec; Manufacturer_No (none) -> TSM-106-01-T-SH
- J18: Manufacturer (none) -> JST; Manufacturer_No (none) -> SM05B-SRSS-TB(LF)(SN)
- J20: Manufacturer (none) -> JST; Manufacturer_No (none) -> SM04B-SRSS-TB(LF)(SN)
- J21: Manufacturer (none) -> Harwin; Manufacturer_No (none) -> M22-5320305
- J4: Arrow Part Number 09452812561 -> (none); Arrow Price/Stock https://www.arrow.com/en/products/09452812561/harting?regio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 -> (none); Manufacturer_No (none) -> 09452812561; Manufacturer_Part_Number 09452812561 -> (none); Mouser Part Number 617-09452812561 -> (none); Mouser Price/Stock https://www.mouser.co.uk/ProductDetail/HARTING/09452812561?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 -> (none)
- J5: LCSC (none) -> C160404; Manufacturer_No (none) -> SM04B-SRSS-TB(LF)(SN)
- J6: Checked y -> (none); Distributor Digikey -> (none); LCSC (none) -> C160404; Manufacturer_No (none) -> SM04B-SRSS-TB(LF)(SN)
- R21, R74, R78: Checked y -> (none); Distributor Mouser -> (none); LCSC C242160 -> DNP; Manufacturer Panasonic -> (none); Manufacturer_No ERJ2GE0R00X -> DNP
- R30: LCSC C60491 -> C60490; Manufacturer_No (none) -> RC0402FR-0710KL
- R55: value DNP -> 0; Checked y -> (none); Distributor Mouser -> (none); LCSC C242160 -> DNP; Manufacturer Panasonic -> (none); Manufacturer_No ERJ2GE0R00X -> DNP
- R63: LCSC C242160 -> C144757; Manufacturer Panasonic -> Yageo; Manufacturer_No ERJ2GE0R00X -> AC0402FR-0747KL
- R64: LCSC C242160 -> (none); Manufacturer Panasonic -> (none); Manufacturer_No ERJ2GE0R00X -> (none)
- R73: LCSC (none) -> C144757; Manufacturer_No (none) -> AC0402FR-0747KL
- U12: value AP22815 -> AP22815A; Checked y -> (none); Distributor Mouser -> (none); LCSC C2150272 -> (none)
- U7: Manufacturer (none) -> Texas Instruments; Manufacturer_No (none) -> SN74LVC1G34DCKR
Connections:
- net PHONE_CLK_3V3: now also R74.1, R86.1, R88.1; no longer U1.192 (SAI3_TXC)
- net PHONE_SYNC_3V3: now also R21.1, R55.1; no longer R21.2, R55.2
- net at U1.200 (SAI3_RXC): now also R88.2
- net DAC_RXFS: no longer names the net of U1.168 (SAI2_RXFS)
- net PHONE_RXFS_3V3: no longer names the net of U1.190 (SAI3_TXFS)
- net PHONE_RXFS_3V3: now also R55.2; no longer R55.1
- net PHONE_TXFS_3V3: no longer names the net of U1.198 (SAI3_RXFS)
- net PHONE_TXFS_3V3: now also R21.2; no longer R21.1
- new net: R86.2, U1.192 (SAI3_TXC)
- no-connect marks 188 -> 187
Other:
- note added: "MCLK+BCLK are the same for the modem (CLK). all clocks can be bidrectional."
- note added: "NOTE: substituted 3.16k"
- note added: "TODO: N/P swapped"
- note added: "TODO: missing connection to GPIO?"
- note added: "TODO: ordered B version by accident (active low)"
- moved on the sheet: R21, R55

Commit message: WIP mb audio rerouting
Parts:
- removed C97, C99: 1uF, Capacitor_SMD:C_0402_1005Metric, symbol Device:C_Small
- removed C98: 10uF, Capacitor_SMD:C_0402_1005Metric, symbol Device:C_Small
- removed R71: 0, Resistor_SMD:R_0402_1005Metric, symbol Device:R_Small
- removed U9: TUSB8040PFP, footprints:QFP50P1400X1400X120-81N, symbol pocket-reform:TUSB8040PFP
- added C38: 0.1uF, Capacitor_SMD:C_0402_1005Metric, symbol Device:C_Small
- added FB11: 220@100MHz 1.4A, Inductor_SMD:L_0603_1608Metric, symbol Device:FerriteBead_Small
- added FB12, FB13: 100@100MHz 3A, Inductor_SMD:L_0603_1608Metric, symbol Device:FerriteBead_Small
- added R101, R95: 4.7k, Resistor_SMD:R_0402_1005Metric, symbol Device:R_Small
- added U25: TUSB8041, Package_DFN_QFN:QFN-64-1EP_9x9mm_P0.5mm_EP6x6mm_ThermalVias, symbol Interface_USB:TUSB8041
- C94: value 0.1uF -> 10uF; LCSC C1525 -> C315248; Manufacturer_No CL05B104KO5NNNC -> CL05A106MP5NUNC
- C95: value 1uF -> 0.1uF; LCSC C14445 -> C1525; Manufacturer_No CL05A105KP5NNNC -> CL05B104KO5NNNC
- C96: value 0.1uF -> DNP
- R23: value 9.09K 1% -> 9.53K 1%; LCSC C400642 -> (none); Manufacturer Panasonic -> (none); Manufacturer_No ERJ2RKF9091X -> (none)
- R25: value 10k -> 4.7k; LCSC C60490 -> C105871; Manufacturer_No RC0402FR-0710KL -> RC0402FR-074K7L
- R63: value 47k -> 0; LCSC C144757 -> C242160; Manufacturer Yageo -> Panasonic; Manufacturer_No AC0402FR-0747KL -> ERJ2GE0R00X
Connections:
- net +1V1: now also FB11.2; no longer C1.1, C100.1, C101.1, C3.1, C70.1, C71.1, C74.1, C79.1, C81.1, C94.1, C96.1
- net +1V8: now also FB12.1; no longer C56.1, C62.1, R70.2, U18.3 (DVDD)
- net +3V3: now also R24.1, R26.1, FB13.2
- net AUD_3V3: now also J18.1 (Pin_1); no longer R63.2
- net GND: now also C21.2, C23.2, C95.1, R23.1, R63.2, Y1.2, Y1.4, C38.2, R101.1, R95.1, U25.65 (VSS); no longer C50.2, C51.2, C57.2, C67.2, C76.2, C78.2, C95.2, C96.2, J18.5 (Pin_5), R25.2, U18.16 (AVSS), U18.20 (SPKVSS), U18.25 (SPKVSS), U18.29 (HPVSS), U18.33 (EP)
- net HEAD_MIC: now also C96.2
- net IMX_UART1_RX: now also R26.2
- net IMX_UART2_RX: now also R24.2
- net USB1_DN: now also U25.54 (USB_DM_UP)
- net USB1_DP: now also U25.53 (USB_DP_UP)
- net USB1_RXN: now also U25.56 (USB_SSTXM_UP)
- net USB1_RXP: now also U25.55 (USB_SSTXP_UP)
- net USB1_TXN: now also U25.59 (USB_SSRXM_UP)
- net USB1_TXP: now also U25.58 (USB_SSRXP_UP)
- net USBH_1A_RXN: now also U25.7 (USB_SSRXM_DN1)
- net USBH_1A_RXP: now also U25.6 (USB_SSRXP_DN1)
- net USBH_1A_TXN: now also U25.4 (USB_SSTXM_DN1)
- net USBH_1A_TXP: now also U25.3 (USB_SSTXP_DN1)
- net USBH_1B_RXN: now also U25.22 (USB_SSRXP_DN3)
- net USBH_1B_RXP: now also U25.23 (USB_SSRXM_DN3)
- net USBH_1B_TXN: now also U25.19 (USB_SSTXP_DN3)
- net USBH_1B_TXP: now also U25.20 (USB_SSTXM_DN3)
- net USBH_1_DN: now also U25.2 (USB_DM_DN1)
- net USBH_1_DP: now also U25.1 (USB_DP_DN1)
- net USBH_2A_RXN: now also U25.15 (USB_SSRXM_DN2)
- net USBH_2A_RXP: now also U25.14 (USB_SSRXP_DN2)
- net USBH_2A_TXN: now also U25.12 (USB_SSTXM_DN2)
- net USBH_2A_TXP: now also U25.11 (USB_SSTXP_DN2)
- net USBH_2B_RXN: now also U25.29 (USB_SSRXP_DN4)
- net USBH_2B_RXP: now also U25.30 (USB_SSRXM_DN4)
- net USBH_2B_TXN: now also U25.26 (USB_SSTXP_DN4)
- net USBH_2B_TXP: now also U25.27 (USB_SSTXM_DN4)
- net USBH_2_DN: now also U25.10 (USB_DM_DN2)
- net USBH_2_DP: now also U25.9 (USB_DP_DN2)
- net USBH_3V3: now also C94.1, R25.2, C38.1, U25.16 (VDD33), U25.34 (VDD33), U25.52 (VDD33), U25.63 (VDD33); no longer C95.1, R24.1, R26.1
- net USBH_3_DN: now also U25.18 (USB_DM_DN3)
- net USBH_3_DP: now also U25.17 (USB_DP_DN3)
- net USBH_4_DN: now also U25.25 (USB_DM_DN4)
- net USBH_4_DP: now also U25.24 (USB_DP_DN4)
- net at U18.2 (IOVDD): now also C95.2, FB13.1
- net at R5.1: now also U25.50 (GRSTz)
- net GNDA: now reaches R63.1
- net GNDA: now also C50.2, C51.2, C57.2, C67.2, C76.2, C78.2, C96.1, J18.5 (Pin_5), U18.16 (AVSS), U18.20 (SPKVSS), U18.25 (SPKVSS), U18.29 (HPVSS), U18.33 (EP); no longer J18.1 (Pin_1)
- net at R22.1, R3.2: now also U25.48 (USB_VBUS)
- net at R25.1: now also U25.40 (FULLPWRMGMTz/SMBA1/SS_UP)
- net at C21.1, R2.1, Y1.1: now also U25.61 (XO)
- net at C23.1, R2.2, Y1.3: now also U25.62 (XI)
- net at R23.2: now also U25.64 (USB_R1)
- new net: C56.1, C62.1, FB12.2, R70.2, U18.3 (DVDD)
- new net: R95.2, U25.49 (TEST)
- new net: R101.2, U25.42 (GANGED/SMBA2/HS_UP)
- new net USBH_1V1: C1.1, C100.1, C101.1, C3.1, C70.1, C71.1, C74.1, C79.1, C81.1, FB11.1, U25.13 (VDD), U25.21 (VDD), U25.28 (VDD), U25.31 (VDD), U25.5 (VDD), U25.51 (VDD), U25.57 (VDD), U25.8 (VDD)
- no-connect marks 187 -> 192
Other:
- note removed: "NOTE: TX/RX were swapped in D-1"
- note removed: "TODO: missing connection to GPIO?"
- note removed: "alt: USB5534B-5000JZX"
- note removed: "alt: USB7200"
- note removed: "disables U1/U2 states NOTE: possibly control by LPC"
- moved on the sheet: C1, C101, C21, C23, C3, C56, C62, C70, C71, C74, C78, C79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

Commit message: motherboard: R-1
Parts:
- removed R31, R32, R49, R51, R63: 0, Resistor_SMD:R_0402_1005Metric, symbol Device:R_Small
- added C106: 22uF, Capacitor_SMD:C_0805_2012Metric, symbol Device:C_Small
- added C107, C98: 10uF, Capacitor_SMD:C_0603_1608Metric, symbol Device:C_Small
- added C108, C109, C97, C99: 0.1uF, Capacitor_SMD:C_0402_1005Metric, symbol Device:C_Small
- added FB14, FB15, FB16: 100@100MHz 3A, Inductor_SMD:L_0603_1608Metric, symbol Device:FerriteBead_Small
- added J17: POWSW, Connector_JST:JST_SH_SM02B-SRSS-TB_1x02-1MP_P1.00mm_Horizontal, symbol Connector:Conn_01x02_Pin
- added U26: 74HC573, Package_SO:TSSOP-20_4.4x6.5mm_P0.65mm, symbol 74xx:74LS573
- added U9: TPS7A0533PDBZ, Package_TO_SOT_SMD:SOT-23, symbol Regulator_Linear:TPS7A0533PDBZ
- C102, C103: footprint Capacitor_SMD:C_0805_2012Metric -> Capacitor_SMD:C_1206_3216Metric; Manufacturer Taiyo Yuden -> (none); Manufacturer_No JMK212BBJ476MG-T -> (none)
- C67: value 10uF -> 22uF; footprint Capacitor_SMD:C_0603_1608Metric -> Capacitor_SMD:C_0805_2012Metric; LCSC C92487 -> (none); Manufacturer_No CL10A106MO8NQNC -> (none)
- FB5: value 100@100MHz 3A -> DNP
- U7: footprint Package_TO_SOT_SMD:SOT-23-5 -> Package_TO_SOT_SMD:SOT-353_SC-70-5
Connections:
- net +5V: now also C108.1, U9.3 (VI)
- net 1V1_ENABLE: now also U8.35 (GPIO23), U26.4 (D2); no longer R46.2, R8.1, U3.4 (EN)
- net 3V3_ENABLE: now also U8.36 (GPIO24), U26.3 (D1); no longer R7.1, U6.5 (EN)
- net 5V_ENABLE: now also U8.37 (GPIO25), U26.2 (D0); no longer R6.1, U5.5 (EN)
- net AUD_3V3: now also C107.1, C97.1, U9.2 (VO)
- net DISP_EN: now also U8.9 (GPIO7), U26.6 (D4); no longer J13.2 (Pin_2)
- net GND: now also R46.2, C108.2, C109.2, C98.2, FB14.1, FB15.1, FB16.1, J17.1 (Pin_1), U26.10 (GND), U9.1 (GND)
- net GNDA: now also C106.2, C107.2, C97.2, C99.2, FB14.2, FB15.2, FB16.2
- net RUD+: now also J21.4 (Pin_4); no longer J21.6 (Pin_6)
- net RUD-: now also J21.3 (Pin_3); no longer J21.5 (Pin_5)
- net STANDBY_3V3: now also C109.1, U26.20 (VCC)
- net XUD+: now also J21.6 (Pin_6); no longer J21.4 (Pin_4)
- net XUD-: now also J21.5 (Pin_5); no longer J21.3 (Pin_3)
- net ~{DISP_RESET}: now also U8.4 (GPIO2), U26.5 (D3); no longer R20.1, U7.2
- net ~{STANDBY_SHDN}: now also J17.2 (Pin_2)
- net at C95.2, FB13.1, U18.2 (IOVDD): now also C98.1
- net at C57.1, C67.1, FB2.2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: now also C106.1, C99.1
- net at R46.1: now also U26.1 (OE); no longer U8.35 (GPIO23)
- net PWREN_LATCH: now reaches U8.41 (GPIO29_ADC3)
- net PWREN_LATCH: now also U26.11 (Load)
- new net: R6.1, U26.19 (Q0), U5.5 (EN)
- new net: R7.1, U26.18 (Q1), U6.5 (EN)
- new net: R8.1, U26.17 (Q2), U3.4 (EN)
- new net DISP_EN_L: J13.2 (Pin_2), U26.15 (Q4)
- new net ~{DISP_RESET_L}: R20.1, U26.16 (Q3), U7.2
- no-connect marks 192 -> 197
Other:
- note added: "Hard Powerdown Interface"
- note added: "Latch for Enables"
- note added: "TODO: test which of these are required"
- note removed: "NOTE: substituted 3.16k"
- note removed: "Temp monitor?"
- moved on the sheet: C17, C50, C56, C6, C62, C67, C95, D3, FB13, FB2, FB5, J20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

Commit message: update motherboard pcb
Parts:
- C102, C103: LCSC (none) -> C94034; Manufacturer (none) -> Murata; Manufacturer_No (none) -> GRM31CR61A476ME15L
- C106, C67: LCSC (none) -> C86295; Manufacturer_No (none) -> CL10A226MP8NUNE
- H5, H7: LCSC C2915626 -> (none); Manufacturer_No SMTSO2020CTJ -> 9774020243R
- H8, H9: LCSC C2915626 -> (none); Manufacturer Sinhoo -> Wurth; Manufacturer_No SMTSO2020CTJ -> 9774025243R
- J17: Manufacturer (none) -> JST; Manufacturer_No (none) -> SM02B-SRSS-TB(LF)(SN)
- R21, R62, R74, R78, R88, TP5, TP6: Manufacturer (none) -> DNP
- R23: LCSC (none) -> C321660; Manufacturer (none) -> FH; Manufacturer_No (none) -> RC-02W9531FT
- R55, R86: value 0 -> 33; Manufacturer (none) -> DNP
- R64: LCSC (none) -> C114762; Manufacturer (none) -> Yageo; Manufacturer_No (none) -> RC0402FR-072K2L
- U12: LCSC (none) -> C2150007
- U25: Manufacturer (none) -> Texas Instruments; Manufacturer_No (none) -> TUSB8041
- U26: LCSC (none) -> C5944
- U7: LCSC (none) -> C7394031; Manufacturer Texas Instruments -> Texas Instruments or UMW
- U9: Manufacturer (none) -> Texas Instruments; Manufacturer_No (none) -> TPS7A0533PDBZ
Connections:
- no-connect marks 197 -> 198
Other:
- note added: "Heatsink/SOM Mount"
- note added: "N/P swapped"
- note added: "WARNING: do not use B version by accident (active low)"
- note removed: "Heatsink Mount"
- note removed: "TODO: N/P swapped"
- note removed: "TODO: ordered B version by accident (active low)"

Commit message: various kicad bumps
Parts:
- J12: Manufacturer_No 1-2199230-5 -> 2199230-5
Other:
- note added: "Alt: Foxconn AS0BC21-S40BB-7H"
- note added: "NOT 1-2199230-5!"
- note added: "Not connected"
Changed lines of the file:
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@@
     (effects (font (size 1.27 1.27)) (justify left bottom))
   )
+  (text "NOT 1-2199230-5!" (at 737.87 359.41 0)
+    (effects (font (size 1.27 1.27)) (justify left bottom))
+  )
   (text "MAX 24V" (at 167.64 106.68 0)
     (effects (font (size 1.27 1.27)) (justify left bottom))
@@
     (effects (font (size 1.27 1.27)) (justify left bottom))
   )
+  (text "Alt: Foxconn AS0BC21-S40BB-7H" (at 730.25 361.95 0)
+    (effects (font (size 1.27 1.27)) (justify left bottom))
+  )
   (text "rated to 28V" (at 866.14 74.93 0)
     (effects (font (size 1.27 1.27)) (justify left bottom))
@@
     (effects (font (size 1.27 1.27)) (justify left bottom))
   )
+  (text "Not connected" (at 266.7 402.59 0)
+    (effects (font (size 1.27 1.27)) (justify left bottom))
+  )
   (text "Includes ESD protection" (at 937.26 556.26 0)
     (effects (font (size 1.27 1.27)) (justify left bottom))
@@
       (effects (font (size 1.27 1.27)) hide)
     )
-    (property "Manufacturer_No" "1-2199230-5" (at 746.76 417.83 0)
+    (property "Manufacturer_No" "2199230-5" (at 746.76 417.83 0)
       (effects (font (size 1.27 1.27)) hide)
     )
