File: pocket-reform-keyboard-kailh-ortho/pocket-reform-keyboard-kailh-ortho.kicad_sch (KiCad schematic)
At the start: 128 parts, among them SW1 Choc, SW10 Choc, SW11 Choc, SW12 Choc, SW13 Choc, SW14 Choc, SW15 Choc, SW16 Choc, SW17 Choc, SW18 Choc, SW19 Choc, SW2 Choc, SW20 Choc, SW21 Choc, SW22 Choc, SW23 Choc, SW24 Choc, SW25 Choc, SW26 Choc, SW27 Choc, SW28 Choc, SW29 Choc, SW3 Choc, SW30 Choc, SW31 Choc, SW32 Choc, SW33 Choc, SW34 Choc, SW35 Choc, SW36 Choc, SW37 Choc, SW38 Choc, SW39 Choc, SW4 Choc, SW40 Choc, SW41 Choc, SW42 Choc, SW43 Choc, SW44 Choc, SW45 Choc, SW46 Choc, SW47 Choc, SW48 Choc, SW49 Choc, SW5 Choc, SW50 Choc, SW51 Choc, SW52 Choc, SW53 Choc, SW54 Choc, SW55 Choc, SW56 Choc, SW57 Choc, SW58 Choc, SW59 Choc, SW6 Choc, SW60 Choc, SW61 Choc, SW62 Choc, SW63 Choc, SW64 Choc, SW7 Choc, SW8 Choc, SW9 Choc

Commit message: keyboard: add D-1 version (beware, has hw bugs)
Parts:
- D1, D10, D11, D12, D121, D122, D123, D124, D13, D14, D15, D16, D17, D18, D19, D2, D20, D21, D22, D23, D24, D25, D26, D27, D28, D29, D3, D30, D31, D32, D33, D34, D35, D36, D37, D38, D39, D4, D40, D41, D42, D43, D44, D45, D46, D47, D48, D49, D5, D50, D51, D52, D53, D54, D55, D56, D57, D58, D59, D6, D60, D7, D8, D9: LCSC (none) -> C193404
- SW1, SW10, SW11, SW12, SW13, SW14, SW15, SW16, SW17, SW18, SW19, SW2, SW20, SW21, SW22, SW23, SW24, SW25, SW26, SW27, SW28, SW29, SW3, SW30, SW31, SW32, SW33, SW34, SW35, SW36, SW37, SW38, SW39, SW4, SW40, SW41, SW42, SW43, SW44, SW45, SW46, SW47, SW48, SW49, SW5, SW50, SW51, SW52, SW53, SW54, SW55, SW56, SW57, SW58, SW59, SW6, SW60, SW61, SW62, SW63, SW64, SW7, SW8, SW9: LCSC (none) -> C400231
