File: pocket-reform-keyboard-kailh-ortho/pocket-reform-kbd-mcu.kicad_sch (KiCad schematic)
At the start: 177 parts, among them J1 Conn_01x06_Female, J2 USB, J3 UART, J4 AUX, SW65 SW_HWB, SW66 SW_RST, U1 SN74LV1T34DCK, U2 RP2040, U3 W25Q32JVSS, U4 MCP1700-3302E_SOT23, Y1 12MHz 18pF

Commit message: update keyboard pcb
Parts:
- GFX2: footprint footprints:mpre-keyboard-badge-d3 -> footprints:mpre-keyboard-badge-r1
- R8: value 0 -> DNP
- SW65: footprint Button_Switch_SMD:SW_DIP_SPSTx01_Slide_6.7x4.1mm_W6.73mm_P2.54mm_LowProfile_JPin -> footprints:Diptronics-PTLP2; LCSC C402914 -> C318893; Manufacturer Dongguan Guangzhu -> XKB; Manufacturer_No DSIC01LSGET -> TS-1185EC-C-D-B
- U4: Flags (none) -> DNP; LCSC C39051 -> DNP
Other:
- note added: "DNP!"
Changed lines of the file:
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@@
     (effects (font (size 1.524 1.524)) (justify left bottom))
   )
+  (text "DNP!" (at 130.81 251.46 0)
+    (effects (font (size 1.27 1.27)) (justify left bottom))
+  )
   (text "To SYSCTL" (at 201.93 248.92 0)
     (effects (font (size 1.524 1.524)) (justify left bottom))
@@
       (effects (font (size 1.27 1.27)) hide)
     )
-    (property "Flags" "" (at 133.35 259.08 0)
+    (property "Flags" "DNP" (at 133.35 259.08 0)
       (effects (font (size 1.27 1.27)) hide)
     )
-    (property "LCSC" "C39051" (at 133.35 259.08 0)
+    (property "LCSC" "DNP" (at 133.35 259.08 0)
       (effects (font (size 1.27 1.27)) hide)
     )
@@
       (effects (font (size 1.27 1.27)))
     )
-    (property "Value" "0" (at 143.51 261.493 90)
+    (property "Value" "DNP" (at 143.51 261.493 90)
       (effects (font (size 1.27 1.27)))
     )
@@
       (effects (font (size 1.27 1.27)) (justify left))
     )
-    (property "Footprint" "footprints:mpre-keyboard-badge-d3" (at 101.6 271.78 0)
+    (property "Footprint" "footprints:mpre-keyboard-badge-r1" (at 101.6 271.78 0)
       (effects (font (size 1.27 1.27)) hide)
     )
@@
       (effects (font (size 1.27 1.27)) (justify left))
     )
-    (property "Footprint" "Button_Switch_SMD:SW_DIP_SPSTx01_Slide_6.7x4.1mm_W6.73mm_P2.54mm_LowProfile_JPin" (at 66.04 237.49 0)
+    (property "Footprint" "footprints:Diptronics-PTLP2" (at 66.04 237.49 0)
       (effects (font (size 1.27 1.27)) hide)
     )
@@
       (effects (font (size 1.27 1.27)) hide)
     )
-    (property "Manufacturer" "Dongguan Guangzhu" (at 66.04 237.49 0)
+    (property "Manufacturer" "XKB" (at 66.04 237.49 0)
       (effects (font (size 1.27 1.27)) hide)
     )
-    (property "Manufacturer_No" "DSIC01LSGET" (at 66.04 237.49 0)
+    (property "Manufacturer_No" "TS-1185EC-C-D-B" (at 66.04 237.49 0)
       (effects (font (size 1.27 1.27)) hide)
     )
-    (property "LCSC" "C402914" (at 66.04 237.49 0)
+    (property "LCSC" "C318893" (at 66.04 237.49 0)
       (effects (font (size 1.27 1.27)) hide)
     )
