File: pocket-reform-charger/pocket-reform-charger.kicad_pcb (KiCad board)
At the start: 2 copper layers, 33 x 65.5 mm, 67 parts, among them J1 CHARGER, J2 CONN_TH1, J3 CONN_TH2, J4 CONN_TH3, Q1 IRF7458TRPBF, Q2 IRF7458TRPBF, U1 MP2762A, U2 MAX17320G

Commit message: snapshot before change to MP2650
Parts:
- removed H4: MountingHole, MountingHole:MountingHole_2.2mm_M2
- removed J2: CONN_TH1, Connector_JST:JST_PH_S2B-PH-SM4-TB_1x02-1MP_P2.00mm_Horizontal
- removed J3: CONN_TH2, Connector_JST:JST_PH_S2B-PH-SM4-TB_1x02-1MP_P2.00mm_Horizontal
- removed J4: CONN_TH3, Connector_JST:JST_PH_S2B-PH-SM4-TB_1x02-1MP_P2.00mm_Horizontal
- C16, C21, C22: value 0.47uF -> 470nF
- U2: value MAX17320G -> MAX17320G20+
- moved TH2 25.5 mm to (120.2, 109.5)
- moved TH1 18.6 mm to (80.8, 108.0), turned to 90 degrees
- moved TH3 16.5 mm to (80.8, 111.1), turned to -90 degrees
Routing:
- net Net-(U1-NTC): track 15.7 -> 40.4 mm
- net PACKGND: track 16.1 -> 26.2 mm, vias 26 -> 37
- net Net-(U2-TH1): track 23.1 -> 29.5 mm, vias 3 -> 2
- net GND: track 53.1 -> 56.7 mm, vias 23 -> 39
Other:
- board size 33 x 65.5 mm -> 41 x 65.5 mm

Commit message: update charger pcb
Parts:
- removed L2: 1.5uH, Inductor_SMD:L_Sunlord_MWSA0518_5.4x5.2mm
- removed TP3: TestPoint, TestPoint:TestPoint_Pad_1.0x1.0mm
- added C23: 22uF, Capacitor_SMD:C_0805_2012Metric, F.Cu at (111.7, 94.9)
- added R21: 14.7k, Resistor_SMD:R_0603_1608Metric, F.Cu at (100.6, 96.1)
- U1: value MP2762A -> MP2650
- moved H5 3.62 mm to (87.7, 83.7)
- moved TP4 2.20 mm to (102.8, 100.0)
- moved L1 1.12 mm to (109.7, 86.5), turned to -90 degrees
- moved C5 0.48 mm to (104.4, 84.1), turned to -90 degrees
- moved TP1 0.07 mm to (105.0, 100.0)
Routing:
- net Net-(U1-CP1): track 20.1 -> 9.38 mm, vias 0 -> 2
- net Net-(U1-SW2): track 26.9 -> 19.4 mm
- net Net-(U1-PSYS): track 9.30 -> 3.88 mm
- net SYSPOWER: track 58.9 -> 53.9 mm
- net Net-(U2-TH2): track 20.2 -> 18.3 mm
- net I2C_SCL: track 41.1 -> 39.4 mm
- net Net-(U1-SW1): track 7.82 -> 9.55 mm
- net Net-(U2-ALRT): track 3.17 -> 4.58 mm
- net Net-(U1-IBM): track 11.5 -> 10.8 mm
- net Net-(U1-CP2): track 3.92 -> 4.56 mm
- net PACKGND: vias 37 -> 39
- net GND: vias 39 -> 57

Commit message: various kicad bumps
Parts:
- F1: value Fuse_Small -> 1206L300/12SLYR
- TH1: value DNP -> 100k B4700
- TH2, TH3: value DNP -> 10k
