File: pocket-reform-charger/pocket-reform-charger.kicad_sch (KiCad schematic)
At the start: 67 parts, among them J1 CHARGER, J2 CONN_TH1, J3 CONN_TH2, J4 CONN_TH3, Q1 IRF7458TRPBF, Q2 IRF7458TRPBF, U1 MP2762A, U2 MAX17320G20+

Commit message: snapshot before change to MP2650
Parts:
- removed H4: MountingHole, MountingHole:MountingHole_2.2mm_M2, symbol Mechanical:MountingHole
- removed J2: CONN_TH1, Connector_JST:JST_PH_S2B-PH-SM4-TB_1x02-1MP_P2.00mm_Horizontal, symbol Connector_Generic:Conn_01x02
- removed J3: CONN_TH2, Connector_JST:JST_PH_S2B-PH-SM4-TB_1x02-1MP_P2.00mm_Horizontal, symbol Connector_Generic:Conn_01x02
- removed J4: CONN_TH3, Connector_JST:JST_PH_S2B-PH-SM4-TB_1x02-1MP_P2.00mm_Horizontal, symbol Connector_Generic:Conn_01x02
Other:
- note added: "TODO: fuse was too weak"

Commit message: update charger pcb
Parts:
- removed L2: 1.5uH, Inductor_SMD:L_Sunlord_MWSA0518_5.4x5.2mm, symbol Device:L_Small
- removed TP3: TestPoint, TestPoint:TestPoint_Pad_1.0x1.0mm, symbol Connector:TestPoint
- added C23: 22uF, Capacitor_SMD:C_0805_2012Metric, symbol Device:C_Small
- added R21: 14.7k, Resistor_SMD:R_0603_1608Metric, symbol Device:R_Small
- TH1, TH2, TH3: value DNP -> 100k
- U1: value MP2762A -> MP2650; symbol pocket-reform-charger:MP2762A -> pocket-reform-charger:MP2650
Connections:
- net GND: now also C23.2, R21.1
- net SYSPOWER: now also C23.1
- net at U1.12 (PSYS): now also R21.2
Other:
- note added: "nPackCfg bit 11: 100k: THType = 1 10k: THType = 0"
- note removed: "Mouser"
- note removed: "TODO: EP"
- note removed: "TODO: R15 wrong footprint"
- note removed: "TODO: check GND separation in https://datasheets.maximintegrated.com/en/ds/MAX17320G1EVKIT-MAX17320X2EVKIT.pdf"
- moved on the sheet: C12, C4, C6, C8, L1, TH3

Commit message: various kicad bumps
Parts:
- BT1, BT2: LCSC (none) -> C295747; Manufacturer (none) -> JST; Manufacturer_No (none) -> S2B-PH-SM4-TB
- C17, C18, C19, C20, C3, C9: LCSC (none) -> C385964; Manufacturer (none) -> Taiyo Yuden; Manufacturer_No (none) -> GMK107B7104KAHT
- F1: value Fuse_Small -> 1206L300/12SLYR; LCSC C883133 -> C1512043; Manufacturer BHFUSE -> Littelfuse; Manufacturer_No BSMD1206-150-16V -> 1206L300/12SLYR
- L1: Manufacturer (none) -> Sunlord; Manufacturer_No (none) -> MWSA0518S-1R5MT
- Q1, Q2: Manufacturer (none) -> Infineon; Manufacturer_No (none) -> IRF7458TRPBF
- R19, R20: Manufacturer (none) -> Generic; Manufacturer_No (none) -> 0Ohms 0603
- R21: LCSC (none) -> C100775; Manufacturer (none) -> LIZ; Manufacturer_No (none) -> CR0603FA1472G
- TH1: value 100k -> 100k B4700; LCSC (none) -> C153015; Manufacturer (none) -> Panasonic; Manufacturer_No (none) -> ERTJ1VV104J
- TH2, TH3: value 100k -> 10k; LCSC (none) -> C13564; Manufacturer (none) -> Murata; Manufacturer_No (none) -> NCP18XH103F03RB
- U1: Manufacturer (none) -> MPS; Manufacturer_No (none) -> MP2650
- U2: Manufacturer (none) -> Maxim; Manufacturer_No (none) -> MAX17320G20+
Other:
- note added: "NCP18XH103F03RB"
- note removed: "TODO: fuse was too weak"
Changed lines of the file:
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@@
     (stroke (width 0) (type default))
-  )
-  (text "TODO: fuse was too weak" (at 237.49 146.05 0)
-    (effects (font (size 1.27 1.27)) (justify left bottom))
   )
   (text "MWSA0518S-1R5MT / C408344" (at 124.46 64.77 0)
@@
   )
   (text "C10879" (at 287.02 129.54 0)
+    (effects (font (size 1.27 1.27)) (justify left bottom))
+  )
+  (text "NCP18XH103F03RB " (at 330.2 212.09 0)
     (effects (font (size 1.27 1.27)) (justify left bottom))
   )
@@
       (effects (font (size 1.27 1.27)) hide)
     )
+    (property "LCSC" "C385964" (at 246.38 199.39 0)
+      (effects (font (size 1.27 1.27)) hide)
+    )
+    (property "Manufacturer" "Taiyo Yuden" (at 246.38 199.39 0)
+      (effects (font (size 1.27 1.27)) hide)
+    )
+    (property "Manufacturer_No" "GMK107B7104KAHT" (at 246.38 199.39 0)
+      (effects (font (size 1.27 1.27)) hide)
+    )
     (pin "1")
     (pin "2")
@@
       (effects (font (size 1.27 1.27)))
     )
-    (property "Value" "Fuse_Small" (at 257.81 139.7 0)
+    (property "Value" "1206L300/12SLYR" (at 257.81 139.7 0)
       (effects (font (size 1.27 1.27)))
     )
@@
       (effects (font (size 1.27 1.27)) hide)
     )
-    (property "LCSC" "C883133" (at 257.81 142.24 0)
-      (effects (font (size 1.27 1.27)) hide)
-    )
-    (property "Manufacturer" "BHFUSE" (at 257.81 142.24 0)
-      (effects (font (size 1.27 1.27)) hide)
-    )
-    (property "Manufacturer_No" "BSMD1206-150-16V" (at 257.81 142.24 0)
+    (property "LCSC" "C1512043" (at 257.81 142.24 0)
+      (effects (font (size 1.27 1.27)) hide)
+    )
+    (property "Manufacturer" "Littelfuse" (at 257.81 142.24 0)
+      (effects (font (size 1.27 1.27)) hide)
+    )
+    (property "Manufacturer_No" "1206L300/12SLYR" (at 257.81 142.24 0)
       (effects (font (size 1.27 1.27)) hide)
     )
@@
     )
     (property "Datasheet" "https://datasheets.maximintegrated.com/en/ds/MAX17320.pdf" (at 274.32 185.42 0)
+      (effects (font (size 1.27 1.27)) hide)
+    )
+    (property "Manufacturer" "Maxim" (at 284.48 185.42 0)
+      (effects (font (size 1.27 1.27)) hide)
+    )
+    (property "Manufacturer_No" "MAX17320G20+" (at 284.48 185.42 0)
       (effects (font (size 1.27 1.27)) hide)
     )
@@
       (effects (font (size 1.27 1.27)) hide)
     )
+    (property "Manufacturer" "Infineon" (at 290.83 144.78 0)
+      (effects (font (size 1.27 1.27)) hide)
+    )
+    (property "Manufacturer_No" "IRF7458TRPBF" (at 290.83 144.78 0)
+      (effects (font (size 1.27 1.27)) hide)
+    )
     (pin "1")
     (pin "2")
@@
       (effects (font (size 1.27 1.27)) hide)
     )
+    (property "Manufacturer" "JST" (at 227.33 198.12 0)
+      (effects (font (size 1.27 1.27)) hide)
+    )
+    (property "Manufacturer_No" "S2B-PH-SM4-TB" (at 227.33 198.12 0)
+      (effects (font (size 1.27 1.27)) hide)
+    )
+    (property "LCSC" "C295747" (at 227.33 198.12 0)
+      (effects (font (size 1.27 1.27)) hide)
+    )
     (pin "1")
     (pin "2")
@@
       (effects (font (size 1.27 1.27)) hide)
     )
+    (property "Manufacturer" "Generic" (at 256.54 200.66 0)
+      (effects (font (size 1.27 1.27)) hide)
+    )
+    (property "Manufacturer_No" "0Ohms 0603" (at 256.54 200.66 0)
+      (effects (font (size 1.27 1.27)) hide)
+    )
     (pin "1")
     (pin "2")
@@
       (effects (font (size 1.27 1.27)) (justify left))
     )
-    (property "Value" "100k" (at 347.98 226.3775 0)
+    (property "Value" "10k" (at 347.98 226.3775 0)
       (effects (font (size 1.27 1.27)) (justify left))
     )
@@
       (effects (font (size 1.27 1.27)) hide)
     )
+    (property "Manufacturer_No" "NCP18XH103F03RB" (at 345.44 224.79 0)
+      (effects (font (size 1.27 1.27)) hide)
+    )
+    (property "Manufacturer" "Murata" (at 345.44 224.79 0)
+      (effects (font (size 1.27 1.27)) hide)
+    )
+    (property "LCSC" "C13564" (at 345.44 224.79 0)
+      (effects (font (size 1.27 1.27)) hide)
+    )
     (pin "1")
     (pin "2")
@@
       (effects (font (size 1.27 1.27)) hide)
     )
+    (property "LCSC" "C385964" (at 102.87 92.71 0)
+      (effects (font (size 1.27 1.27)) hide)
+    )
+    (property "Manufacturer" "Taiyo Yuden" (at 102.87 92.71 0)
+      (effects (font (size 1.27 1.27)) hide)
+    )
+    (property "Manufacturer_No" "GMK107B7104KAHT" (at 102.87 92.71 0)
+      (effects (font (size 1.27 1.27)) hide)
+    )
     (pin "1")
     (pin "2")
@@
       (effects (font (size 1.27 1.27)) hide)
     )
-    (property "LCSC" "" (at 97.79 172.72 0)
-      (effects (font (size 1.27 1.27)) hide)
-    )
-    (property "Manufacturer" "" (at 97.79 172.72 0)
-      (effects (font (size 1.27 1.27)) hide)
-    )
-    (property "Manufacturer_No" "" (at 97.79 172.72 0)
+    (property "LCSC" "C100775" (at 97.79 172.72 0)
+      (effects (font (size 1.27 1.27)) hide)
+    )
+    (property "Manufacturer" "LIZ" (at 97.79 172.72 0)
+      (effects (font (size 1.27 1.27)) hide)
+    )
+    (property "Manufacturer_No" "CR0603FA1472G" (at 97.79 172.72 0)
       (effects (font (size 1.27 1.27)) hide)
     )
@@
       (effects (font (size 1.27 1.27)) hide)
     )
+    (property "LCSC" "C385964" (at 246.38 213.36 0)
+      (effects (font (size 1.27 1.27)) hide)
+    )
+    (property "Manufacturer" "Taiyo Yuden" (at 246.38 213.36 0)
+      (effects (font (size 1.27 1.27)) hide)
+    )
+    (property "Manufacturer_No" "GMK107B7104KAHT" (at 246.38 213.36 0)
+      (effects (font (size 1.27 1.27)) hide)
+    )
     (pin "1")
     (pin "2")
@@
       (effects (font (size 1.27 1.27)) hide)
     )
+    (property "LCSC" "C385964" (at 254 181.61 0)
+      (effects (font (size 1.27 1.27)) hide)
+    )
+    (property "Manufacturer" "Taiyo Yuden" (at 254 181.61 0)
+      (effects (font (size 1.27 1.27)) hide)
+    )
+    (property "Manufacturer_No" "GMK107B7104KAHT" (at 254 181.61 0)
+      (effects (font (size 1.27 1.27)) hide)
+    )
     (pin "1")
     (pin "2")
@@
       (effects (font (size 1.27 1.27)) hide)
     )
+    (property "Manufacturer" "JST" (at 227.33 214.63 0)
+      (effects (font (size 1.27 1.27)) hide)
+    )
+    (property "Manufacturer_No" "S2B-PH-SM4-TB" (at 227.33 214.63 0)
+      (effects (font (size 1.27 1.27)) hide)
+    )
+    (property "LCSC" "C295747" (at 227.33 214.63 0)
+      (effects (font (size 1.27 1.27)) hide)
+    )
     (pin "1")
     (pin "2")
@@
       (effects (font (size 1.27 1.27)) (justify left))
     )
-    (property "Value" "100k" (at 332.74 226.3775 0)
+    (property "Value" "10k" (at 332.74 226.3775 0)
       (effects (font (size 1.27 1.27)) (justify left))
     )
@@
       (effects (font (size 1.27 1.27)) hide)
     )
+    (property "Manufacturer_No" "NCP18XH103F03RB" (at 330.2 224.79 0)
+      (effects (font (size 1.27 1.27)) hide)
+    )
+    (property "Manufacturer" "Murata" (at 330.2 224.79 0)
+      (effects (font (size 1.27 1.27)) hide)
+    )
+    (property "LCSC" "C13564" (at 330.2 224.79 0)
+      (effects (font (size 1.27 1.27)) hide)
+    )
     (pin "1")
     (pin "2")
@@
       (effects (font (size 1.27 1.27)) (justify left))
     )
-    (property "Value" "100k" (at 187.96 176.8475 0)
+    (property "Value" "100k B4700" (at 187.96 176.8475 0)
       (effects (font (size 1.27 1.27)) (justify left))
     )
@@
       (effects (font (size 1.27 1.27)) hide)
     )
+    (property "Manufacturer" "Panasonic" (at 185.42 175.26 0)
+      (effects (font (size 1.27 1.27)) hide)
+    )
+    (property "Manufacturer_No" "ERTJ1VV104J" (at 185.42 175.26 0)
+      (effects (font (size 1.27 1.27)) hide)
+    )
+    (property "LCSC" "C153015" (at 185.42 175.26 0)
+      (effects (font (size 1.27 1.27)) hide)
+    )
     (pin "1")
     (pin "2")
@@
     )
     (property "Datasheet" "~" (at 266.7 147.32 0)
+      (effects (font (size 1.27 1.27)) hide)
+    )
+    (property "LCSC" "C385964" (at 266.7 147.32 0)
+      (effects (font (size 1.27 1.27)) hide)
+    )
+    (property "Manufacturer" "Taiyo Yuden" (at 266.7 147.32 0)
+      (effects (font (size 1.27 1.27)) hide)
+    )
+    (property "Manufacturer_No" "GMK107B7104KAHT" (at 266.7 147.32 0)
       (effects (font (size 1.27 1.27)) hide)
     )
@@
     )
     (property "LCSC" "C10879" (at 278.13 144.78 0)
+      (effects (font (size 1.27 1.27)) hide)
+    )
+    (property "Manufacturer" "Infineon" (at 278.13 144.78 0)
+      (effects (font (size 1.27 1.27)) hide)
+    )
+    (property "Manufacturer_No" "IRF7458TRPBF" (at 278.13 144.78 0)
       (effects (font (size 1.27 1.27)) hide)
     )
@@
       (effects (font (size 1.27 1.27)) hide)
     )
+    (property "Manufacturer" "Generic" (at 252.73 204.47 0)
+      (effects (font (size 1.27 1.27)) hide)
+    )
+    (property "Manufacturer_No" "0Ohms 0603" (at 252.73 204.47 0)
+      (effects (font (size 1.27 1.27)) hide)
+    )
     (pin "1")
     (pin "2")
@@
     )
     (property "Datasheet" "" (at 132.08 118.11 0)
+      (effects (font (size 1.27 1.27)) hide)
+    )
+    (property "Manufacturer" "MPS" (at 139.7 128.27 0)
+      (effects (font (size 1.27 1.27)) hide)
+    )
+    (property "Manufacturer_No" "MP2650" (at 139.7 128.27 0)
       (effects (font (size 1.27 1.27)) hide)
     )
@@
       (effects (font (size 1.27 1.27)) hide)
     )
+    (property "Manufacturer" "Sunlord" (at 139.7 72.39 0)
+      (effects (font (size 1.27 1.27)) hide)
+    )
+    (property "Manufacturer_No" "MWSA0518S-1R5MT" (at 139.7 72.39 0)
+      (effects (font (size 1.27 1.27)) hide)
+    )
     (pin "1")
     (pin "2")
@@
       (effects (font (size 1.27 1.27)) hide)
     )
+    (property "LCSC" "C385964" (at 180.34 93.98 0)
+      (effects (font (size 1.27 1.27)) hide)
+    )
+    (property "Manufacturer" "Taiyo Yuden" (at 180.34 93.98 0)
+      (effects (font (size 1.27 1.27)) hide)
+    )
+    (property "Manufacturer_No" "GMK107B7104KAHT" (at 180.34 93.98 0)
+      (effects (font (size 1.27 1.27)) hide)
+    )
