File: pocket-reform-headphones/pocket-reform-headphones.kicad_pcb (KiCad board)
At the start: 2 copper layers, 17.6 x 95 mm, 15 parts, among them J1 CONN_HEAD, J2 SJ-43516-SMT, J4 CONN_PWRSW, SW1 SW_DIP_x01

Commit message: various kicad bumps
Parts:
- C2, C3, C4: value 0.1uF -> DNP
- R2, R3, R4: value 220 -> 0
Changed lines of the file:
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@@
       (disableapertmacros false)
       (usegerberextensions false)
-      (usegerberattributes true)
+      (usegerberattributes false)
       (usegerberadvancedattributes true)
       (creategerberjobfile true)
@@
       (drillshape 0)
       (scaleselection 1)
-      (outputdirectory "pref-headset-r1")
+      (outputdirectory "pref-headset-r1b")
     )
   )
@@
     (descr "JST SH series connector, SM05B-SRSS-TB (http://www.jst-mfg.com/product/pdf/eng/eSH.pdf), generated with kicad-footprint-generator")
     (tags "connector JST SH top entry")
+    (property "LCSC" "C136657")
     (property "Manufacturer" "JST")
     (property "Manufacturer_No" "SM05B-SRSS-TB(LF)(SN)")
@@
     (descr "Capacitor SMD 0603 (1608 Metric), square (rectangular) end terminal, IPC_7351 nominal, (Body size source: IPC-SM-782 page 76, https://www.pcb-3d.com/wordpress/wp-content/uploads/ipc-sm-782a_amendment_1_and_2.pdf), generated with kicad-footprint-generator")
     (tags "capacitor")
+    (property "LCSC" "DNP")
+    (property "Manufacturer" "DNP")
+    (property "Manufacturer_No" "DNP")
     (property "Sheetfile" "pocket-reform-headphones.kicad_sch")
     (property "Sheetname" "")
@@
         (effects (font (size 1 1) (thickness 0.15)))
     )
-    (fp_text value "0.1uF" (at 0 1.43) (layer "F.Fab")
+    (fp_text value "DNP" (at 0 1.43) (layer "F.Fab")
         (effects (font (size 1 1) (thickness 0.15)))
     )
@@
     (descr "Resistor SMD 0603 (1608 Metric), square (rectangular) end terminal, IPC_7351 nominal, (Body size source: IPC-SM-782 page 72, https://www.pcb-3d.com/wordpress/wp-content/uploads/ipc-sm-782a_amendment_1_and_2.pdf), generated with kicad-footprint-generator")
     (tags "resistor")
+    (property "LCSC" "")
+    (property "Manufacturer" "Generic")
+    (property "Manufacturer_No" "0Ohms 0603")
     (property "Sheetfile" "pocket-reform-headphones.kicad_sch")
     (property "Sheetname" "")
@@
         (effects (font (size 1 1) (thickness 0.15)))
     )
-    (fp_text value "220" (at 0 1.43) (layer "F.Fab")
+    (fp_text value "0" (at 0 1.43) (layer "F.Fab")
         (effects (font (size 1 1) (thickness 0.15)))
     )
@@
     (descr "Mounting Hole 2.2mm, M2, DIN965")
     (tags "mounting hole 2.2mm m2 din965")
+    (property "LCSC" "")
     (property "Sheetfile" "pocket-reform-headphones.kicad_sch")
     (property "Sheetname" "")
@@
     (property "Checked" "y")
     (property "Distributor" "Mouser")
+    (property "LCSC" "")
     (property "Manufacturer" "CUI")
     (property "Manufacturer_No" "SJ-43516-SMT-TR")
@@
     (property "Checked" "y")
     (property "Distributor" "Mouser")
-    (property "Manufacturer" "Littelfuse")
-    (property "Manufacturer_No" "SP0503BAHT")
+    (property "LCSC" "C3040626")
+    (property "Manufacturer" "Littelfuse / TECH PUBLIC")
+    (property "Manufacturer_No" "SP0503BAHTG")
     (property "Sheetfile" "pocket-reform-headphones.kicad_sch")
     (property "Sheetname" "")
@@
     (descr "Resistor SMD 0603 (1608 Metric), square (rectangular) end terminal, IPC_7351 nominal, (Body size source: IPC-SM-782 page 72, https://www.pcb-3d.com/wordpress/wp-content/uploads/ipc-sm-782a_amendment_1_and_2.pdf), generated with kicad-footprint-generator")
     (tags "resistor")
+    (property "LCSC" "")
+    (property "Manufacturer" "Generic")
+    (property "Manufacturer_No" "0Ohms 0603")
     (property "Sheetfile" "pocket-reform-headphones.kicad_sch")
     (property "Sheetname" "")
@@
         (effects (font (size 1 1) (thickness 0.15)))
     )
-    (fp_text value "220" (at 0 1.43) (layer "F.Fab")
+    (fp_text value "0" (at 0 1.43) (layer "F.Fab")
         (effects (font (size 1 1) (thickness 0.15)))
     )
@@
     (descr "Resistor SMD 0603 (1608 Metric), square (rectangular) end terminal, IPC_7351 nominal, (Body size source: IPC-SM-782 page 72, https://www.pcb-3d.com/wordpress/wp-content/uploads/ipc-sm-782a_amendment_1_and_2.pdf), generated with kicad-footprint-generator")
     (tags "resistor")
+    (property "LCSC" "")
+    (property "Manufacturer" "Generic")
+    (property "Manufacturer_No" "47k 0603")
     (property "Sheetfile" "pocket-reform-headphones.kicad_sch")
     (property "Sheetname" "")
@@
     (descr "Capacitor SMD 0603 (1608 Metric), square (rectangular) end terminal, IPC_7351 nominal, (Body size source: IPC-SM-782 page 76, https://www.pcb-3d.com/wordpress/wp-content/uploads/ipc-sm-782a_amendment_1_and_2.pdf), generated with kicad-footprint-generator")
     (tags "capacitor")
+    (property "LCSC" "DNP")
+    (property "Manufacturer" "DNP")
+    (property "Manufacturer_No" "DNP")
     (property "Sheetfile" "pocket-reform-headphones.kicad_sch")
     (property "Sheetname" "")
@@
         (effects (font (size 1 1) (thickness 0.15)))
     )
-    (fp_text value "0.1uF" (at 0 1.43) (layer "F.Fab")
+    (fp_text value "DNP" (at 0 1.43) (layer "F.Fab")
         (effects (font (size 1 1) (thickness 0.15)))
     )
@@
     (at 89.5 89 -90)
     (descr "Ultraminiature Surface Mount Slide Switch, right-angle, https://www.ckswitches.com/media/1424/pcm.pdf")
+    (property "LCSC" "C319019")
+    (property "Manufacturer" "XKB")
+    (property "Manufacturer_No" "SK-3296S-01-L3")
     (property "Sheetfile" "pocket-reform-headphones.kicad_sch")
     (property "Sheetname" "")
@@
     (descr "Mounting Hole 2.2mm, M2, DIN965")
     (tags "mounting hole 2.2mm m2 din965")
+    (property "LCSC" "")
     (property "Sheetfile" "pocket-reform-headphones.kicad_sch")
     (property "Sheetname" "")
@@
     (descr "JST SH series connector, SM02B-SRSS-TB (http://www.jst-mfg.com/product/pdf/eng/eSH.pdf), generated with kicad-footprint-generator")
     (tags "connector JST SH top entry")
+    (property "LCSC" "C160402")
+    (property "Manufacturer" "JST")
+    (property "Manufacturer_No" "SM02B-SRSS-TB(LF)(SN)")
     (property "Sheetfile" "pocket-reform-headphones.kicad_sch")
     (property "Sheetname" "")
@@
   (footprint "footprints:pref-headset-badge" (layer "F.Cu")
     (at 94.102 119.283834 90)
+    (property "LCSC" "")
     (property "Sheetfile" "pocket-reform-headphones.kicad_sch")
     (property "Sheetname" "")
@@
     (descr "Resistor SMD 0603 (1608 Metric), square (rectangular) end terminal, IPC_7351 nominal, (Body size source: IPC-SM-782 page 72, https://www.pcb-3d.com/wordpress/wp-content/uploads/ipc-sm-782a_amendment_1_and_2.pdf), generated with kicad-footprint-generator")
     (tags "resistor")
+    (property "LCSC" "")
+    (property "Manufacturer" "Generic")
+    (property "Manufacturer_No" "0Ohms 0603")
     (property "Sheetfile" "pocket-reform-headphones.kicad_sch")
     (property "Sheetname" "")
@@
         (effects (font (size 1 1) (thickness 0.15)))
     )
-    (fp_text value "220" (at 0 1.43) (layer "F.Fab")
+    (fp_text value "0" (at 0 1.43) (layer "F.Fab")
         (effects (font (size 1 1) (thickness 0.15)))
     )
@@
     (descr "Capacitor SMD 0603 (1608 Metric), square (rectangular) end terminal, IPC_7351 nominal, (Body size source: IPC-SM-782 page 76, https://www.pcb-3d.com/wordpress/wp-content/uploads/ipc-sm-782a_amendment_1_and_2.pdf), generated with kicad-footprint-generator")
     (tags "capacitor")
+    (property "LCSC" "DNP")
+    (property "Manufacturer" "DNP")
+    (property "Manufacturer_No" "DNP")
     (property "Sheetfile" "pocket-reform-headphones.kicad_sch")
     (property "Sheetname" "")
@@
         (effects (font (size 1 1) (thickness 0.15)))
     )
-    (fp_text value "0.1uF" (at 0 1.43) (layer "F.Fab")
+    (fp_text value "DNP" (at 0 1.43) (layer "F.Fab")
         (effects (font (size 1 1) (thickness 0.15)))
     )
