File: pocket-reform-headphones/pocket-reform-headphones.kicad_sch (KiCad schematic)
At the start: 15 parts, among them J1 CONN_HEAD, J2 SJ-43516-SMT, J4 CONN_PWRSW, SW1 SW_DIP_x01

Commit message: various kicad bumps
Parts:
- C2, C3, C4: value 0.1uF -> DNP; LCSC (none) -> DNP; Manufacturer (none) -> DNP; Manufacturer_No (none) -> DNP
- D1: LCSC (none) -> C3040626; Manufacturer Littelfuse -> Littelfuse / TECH PUBLIC; Manufacturer_No SP0503BAHT -> SP0503BAHTG
- J1: LCSC (none) -> C136657
- J4: LCSC (none) -> C160402; Manufacturer (none) -> JST; Manufacturer_No (none) -> SM02B-SRSS-TB(LF)(SN)
- R1: Manufacturer (none) -> Generic; Manufacturer_No (none) -> 47k 0603
- R2, R3, R4: value 220 -> 0; Manufacturer (none) -> Generic; Manufacturer_No (none) -> 0Ohms 0603
- SW1: LCSC (none) -> C319019; Manufacturer (none) -> XKB; Manufacturer_No (none) -> SK-3296S-01-L3
Other:
- note added: "TODO: confirm R3/R4 ohms"
Changed lines of the file:
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@@
+    (effects (font (size 1.27 1.27)) (justify left bottom))
+  )
+  (text "TODO: confirm R3/R4 ohms" (at 50.8 58.42 0)
     (effects (font (size 1.27 1.27)) (justify left bottom))
   )
@@
       (effects (font (size 1.27 1.27)) hide)
     )
+    (property "LCSC" "" (at 57.15 83.82 0)
+      (effects (font (size 1.27 1.27)) hide)
+    )
     (pin "1")
     (instances
@@
       (effects (font (size 1.27 1.27)) hide)
     )
-    (property "Manufacturer" "Littelfuse" (at 133.35 57.15 0)
-      (effects (font (size 1.27 1.27)) hide)
-    )
-    (property "Manufacturer_No" "SP0503BAHT" (at 133.35 57.15 0)
+    (property "Manufacturer" "Littelfuse / TECH PUBLIC" (at 133.35 57.15 0)
+      (effects (font (size 1.27 1.27)) hide)
+    )
+    (property "Manufacturer_No" "SP0503BAHTG" (at 133.35 57.15 0)
       (effects (font (size 1.27 1.27)) hide)
     )
     (property "Checked" "y" (at 133.35 57.15 0)
+      (effects (font (size 1.27 1.27)) hide)
+    )
+    (property "LCSC" "C3040626" (at 133.35 57.15 0)
       (effects (font (size 1.27 1.27)) hide)
     )
@@
       (effects (font (size 1.27 1.27)))
     )
-    (property "Value" "220" (at 76.2 39.37 90)
+    (property "Value" "0" (at 76.2 39.37 90)
       (effects (font (size 1.27 1.27)))
     )
@@
     )
     (property "Datasheet" "~" (at 76.2 41.91 0)
+      (effects (font (size 1.27 1.27)) hide)
+    )
+    (property "LCSC" "" (at 76.2 41.91 0)
+      (effects (font (size 1.27 1.27)) hide)
+    )
+    (property "Manufacturer" "Generic" (at 76.2 41.91 0)
+      (effects (font (size 1.27 1.27)) hide)
+    )
+    (property "Manufacturer_No" "0Ohms 0603" (at 76.2 41.91 0)
       (effects (font (size 1.27 1.27)) hide)
     )
@@
       (effects (font (size 1.27 1.27)) hide)
     )
+    (property "LCSC" "C136657" (at 36.83 40.64 0)
+      (effects (font (size 1.27 1.27)) hide)
+    )
     (pin "1")
     (pin "2")
@@
       (effects (font (size 1.27 1.27)) hide)
     )
+    (property "LCSC" "" (at 60.96 88.9 0)
+      (effects (font (size 1.27 1.27)) hide)
+    )
     (pin "1")
     (instances
@@
       (effects (font (size 1.27 1.27)))
     )
-    (property "Value" "220" (at 76.2 46.99 90)
+    (property "Value" "0" (at 76.2 46.99 90)
       (effects (font (size 1.27 1.27)))
     )
@@
     )
     (property "Datasheet" "~" (at 76.2 49.53 0)
+      (effects (font (size 1.27 1.27)) hide)
+    )
+    (property "LCSC" "" (at 76.2 49.53 0)
+      (effects (font (size 1.27 1.27)) hide)
+    )
+    (property "Manufacturer" "Generic" (at 76.2 49.53 0)
+      (effects (font (size 1.27 1.27)) hide)
+    )
+    (property "Manufacturer_No" "0Ohms 0603" (at 76.2 49.53 0)
       (effects (font (size 1.27 1.27)) hide)
     )
@@
       (effects (font (size 1.27 1.27)) (justify left))
     )
-    (property "Value" "0.1uF" (at 83.82 57.1563 0)
+    (property "Value" "DNP" (at 83.82 57.1563 0)
       (effects (font (size 1.27 1.27)) (justify left))
     )
@@
       (effects (font (size 1.27 1.27)) hide)
     )
+    (property "LCSC" "DNP" (at 81.28 55.88 0)
+      (effects (font (size 1.27 1.27)) hide)
+    )
+    (property "Manufacturer" "DNP" (at 81.28 55.88 0)
+      (effects (font (size 1.27 1.27)) hide)
+    )
+    (property "Manufacturer_No" "DNP" (at 81.28 55.88 0)
+      (effects (font (size 1.27 1.27)) hide)
+    )
     (pin "1")
     (pin "2")
@@
       (effects (font (size 1.27 1.27)) hide)
     )
+    (property "LCSC" "" (at 41.91 69.85 0)
+      (effects (font (size 1.27 1.27)) hide)
+    )
+    (property "Manufacturer" "Generic" (at 41.91 69.85 0)
+      (effects (font (size 1.27 1.27)) hide)
+    )
+    (property "Manufacturer_No" "47k 0603" (at 41.91 69.85 0)
+      (effects (font (size 1.27 1.27)) hide)
+    )
     (pin "1")
     (pin "2")
@@
     )
     (property "Datasheet" "~" (at 67.31 100.33 0)
+      (effects (font (size 1.27 1.27)) hide)
+    )
+    (property "LCSC" "" (at 67.31 100.33 0)
       (effects (font (size 1.27 1.27)) hide)
     )
@@
       (effects (font (size 1.27 1.27)) (justify left))
     )
-    (property "Value" "0.1uF" (at 104.14 57.1563 0)
+    (property "Value" "DNP" (at 104.14 57.1563 0)
       (effects (font (size 1.27 1.27)) (justify left))
     )
@@
     )
     (property "Datasheet" "~" (at 101.6 55.88 0)
+      (effects (font (size 1.27 1.27)) hide)
+    )
+    (property "LCSC" "DNP" (at 101.6 55.88 0)
+      (effects (font (size 1.27 1.27)) hide)
+    )
+    (property "Manufacturer" "DNP" (at 101.6 55.88 0)
+      (effects (font (size 1.27 1.27)) hide)
+    )
+    (property "Manufacturer_No" "DNP" (at 101.6 55.88 0)
       (effects (font (size 1.27 1.27)) hide)
     )
@@
       (effects (font (size 1.27 1.27)) hide)
     )
+    (property "LCSC" "" (at 144.78 41.91 0)
+      (effects (font (size 1.27 1.27)) hide)
+    )
     (pin "1")
     (pin "2")
@@
       (effects (font (size 1.27 1.27)) (justify left))
     )
-    (property "Value" "0.1uF" (at 93.98 57.1563 0)
+    (property "Value" "DNP" (at 93.98 57.1563 0)
       (effects (font (size 1.27 1.27)) (justify left))
     )
@@
       (effects (font (size 1.27 1.27)) hide)
     )
+    (property "LCSC" "DNP" (at 91.44 55.88 0)
+      (effects (font (size 1.27 1.27)) hide)
+    )
+    (property "Manufacturer" "DNP" (at 91.44 55.88 0)
+      (effects (font (size 1.27 1.27)) hide)
+    )
+    (property "Manufacturer_No" "DNP" (at 91.44 55.88 0)
+      (effects (font (size 1.27 1.27)) hide)
+    )
     (pin "1")
     (pin "2")
@@
       (effects (font (size 1.27 1.27)) hide)
     )
+    (property "LCSC" "C319019" (at 134.62 129.54 0)
+      (effects (font (size 1.27 1.27)) hide)
+    )
+    (property "Manufacturer" "XKB" (at 134.62 129.54 0)
+      (effects (font (size 1.27 1.27)) hide)
+    )
+    (property "Manufacturer_No" "SK-3296S-01-L3" (at 134.62 129.54 0)
+      (effects (font (size 1.27 1.27)) hide)
+    )
     (pin "1")
     (pin "2")
@@
       (effects (font (size 1.27 1.27)))
     )
-    (property "Value" "220" (at 110.49 34.29 90)
+    (property "Value" "0" (at 110.49 34.29 90)
       (effects (font (size 1.27 1.27)))
     )
@@
       (effects (font (size 1.27 1.27)) hide)
     )
+    (property "LCSC" "" (at 110.49 36.83 0)
+      (effects (font (size 1.27 1.27)) hide)
+    )
+    (property "Manufacturer" "Generic" (at 110.49 36.83 0)
+      (effects (font (size 1.27 1.27)) hide)
+    )
+    (property "Manufacturer_No" "0Ohms 0603" (at 110.49 36.83 0)
+      (effects (font (size 1.27 1.27)) hide)
+    )
     (pin "1")
     (pin "2")
@@
       (effects (font (size 1.27 1.27)) hide)
     )
+    (property "LCSC" "C160402" (at 165.1 129.54 0)
+      (effects (font (size 1.27 1.27)) hide)
+    )
+    (property "Manufacturer" "JST" (at 165.1 129.54 0)
+      (effects (font (size 1.27 1.27)) hide)
+    )
+    (property "Manufacturer_No" "SM02B-SRSS-TB(LF)(SN)" (at 165.1 129.54 0)
+      (effects (font (size 1.27 1.27)) hide)
+    )
